File: hardware/pcb-mods/nova_pcb_v6/02_power_rails.kicad_sch (KiCad schematic)
At the start: 8 parts, among them J12 XT30_JET_12V, J13 XT30_L2_12V, J2 UBEC_5V_AUX, U1 Pololu_D42V110F7_LEG_7V5, U2 Pololu_D42V110F12_HIP_12V, U3 Pololu_D24V22F12_L2_12V, U4 Pololu_D42V55F12_JET_12V, U5 Pololu_D42V55F7_ARM_7V5

Commit message: pcb(v6-power-v2): fork to v2 — full reroute, safety chain, off-board INA226, DRC clean
- Fork nova_pcb_v6_power -> _v2 (v1 frozen); placement redone power-flow-first
- Safety chain board sync: Q3 e-stop inverter, Q4 EN_JET cutoff, R16, C8/C9
- INA226 modules converted off-board: footprints stripped to 4-pin I2C headers,
  RAW nets eliminated (bench wiring card in ROUTING_HANDOFF.md Step 8)
- All power routed 1.5/3.0mm per netclass, LEG pour L-shape, hip doubled F+B
- All signal nets routed headless via pre-commit collision checker:
  B.Cu lanes y137.5-139.9 + F.Cu verticals + via pairs; V5_AUX spine gap
  bridged x114.5; board min via relaxed to 0.45/0.25 (PCBWay standard)
- DRC: 0 errors, 0 unrouted; 2 zone-island seams left for GUI (Step 9)

Co-Authored-By: Claude Fable 5 <noreply@anthropic.com>
Parts:
- added C6: 470uF_25V, Capacitor_THT:CP_Radial_D10.0mm_P5.00mm, symbol Device:C
- added L1: 22uH, Inductor_SMD:L_12x12mm_H8mm, symbol Device:L
- U1, U2: footprint Connector_PinHeader_2.54mm:PinHeader_1x04_P2.54mm_Vertical -> nova_v6:Pololu_D42V110Fx
- U3: footprint Connector_PinHeader_2.54mm:PinHeader_1x04_P2.54mm_Vertical -> nova_v6:Pololu_D24V22Fx
- U4, U5: footprint Connector_PinHeader_2.54mm:PinHeader_1x04_P2.54mm_Vertical -> nova_v6:Pololu_D42V55Fx
Connections:
- net GND: now also C6.2
- net V12_HIP: no longer U2.4 (Pin_4)
- net V12_JET: no longer U4.4 (Pin_4)
- net V12_L2: now also C6.1, L1.2; no longer U3.4 (Pin_4)
- net V7V5_LEG: no longer U1.4 (Pin_4)
- new net V12_HIP_RAW: U2.4 (Pin_4)
- new net V12_JET_RAW: U4.4 (Pin_4)
- new net V12_L2_RAW: L1.1, U3.4 (Pin_4)
- new net V7V5_LEG_RAW: U1.4 (Pin_4)
