File: hardware/pcb-mods/nova_pcb_v6/06_safety_chain.kicad_sch (KiCad schematic)
At the start: 17 parts, among them Q2 BSS138_cutoff, SW2 Estop_NC_latching, U10 INA226, U11 INA226, U8 LM393, U9 INA226

Commit message: pcb(v6-power-v2): fork to v2 — full reroute, safety chain, off-board INA226, DRC clean
- Fork nova_pcb_v6_power -> _v2 (v1 frozen); placement redone power-flow-first
- Safety chain board sync: Q3 e-stop inverter, Q4 EN_JET cutoff, R16, C8/C9
- INA226 modules converted off-board: footprints stripped to 4-pin I2C headers,
  RAW nets eliminated (bench wiring card in ROUTING_HANDOFF.md Step 8)
- All power routed 1.5/3.0mm per netclass, LEG pour L-shape, hip doubled F+B
- All signal nets routed headless via pre-commit collision checker:
  B.Cu lanes y137.5-139.9 + F.Cu verticals + via pairs; V5_AUX spine gap
  bridged x114.5; board min via relaxed to 0.45/0.25 (PCBWay standard)
- DRC: 0 errors, 0 unrouted; 2 zone-island seams left for GUI (Step 9)

Co-Authored-By: Claude Fable 5 <noreply@anthropic.com>
Parts:
- R10, R11, R12, R2, R3, R4, R5, R6, R7, R8, R9: now not fitted
- U10, U11, U9: footprint Package_SO:VSSOP-10_3x3mm_P0.5mm -> nova_v6:INA226_Module_Breakout
Connections:
- net V12_HIP: no longer U10.10 (Vin+)
- net V12_JET: no longer U11.10 (Vin+)
- net V7V5_LEG: no longer U9.10 (Vin+)
- new net V12_HIP_RAW: U10.10 (Vin+)
- new net V12_JET_RAW: U11.10 (Vin+)
- new net V7V5_LEG_RAW: U9.10 (Vin+)
