File: hardware/pcb-mods/nova_pcb_v6/nova_pcb_v6.kicad_pcb (KiCad board)
At the start: 4 copper layers, 0 parts

Commit message: pcb(v6-power-v2): fork to v2 — full reroute, safety chain, off-board INA226, DRC clean
- Fork nova_pcb_v6_power -> _v2 (v1 frozen); placement redone power-flow-first
- Safety chain board sync: Q3 e-stop inverter, Q4 EN_JET cutoff, R16, C8/C9
- INA226 modules converted off-board: footprints stripped to 4-pin I2C headers,
  RAW nets eliminated (bench wiring card in ROUTING_HANDOFF.md Step 8)
- All power routed 1.5/3.0mm per netclass, LEG pour L-shape, hip doubled F+B
- All signal nets routed headless via pre-commit collision checker:
  B.Cu lanes y137.5-139.9 + F.Cu verticals + via pairs; V5_AUX spine gap
  bridged x114.5; board min via relaxed to 0.45/0.25 (PCBWay standard)
- DRC: 0 errors, 0 unrouted; 2 zone-island seams left for GUI (Step 9)

Co-Authored-By: Claude Fable 5 <noreply@anthropic.com>
Parts:
- added C1: 1000uF_25V, Capacitor_THT:CP_Radial_D12.5mm_P5.00mm, F.Cu at (18.0, 22.0)
- added C2: 1000uF_25V, Capacitor_THT:CP_Radial_D12.5mm_P5.00mm, F.Cu at (18.0, 36.0)
- added C3: 1000uF_25V, Capacitor_THT:CP_Radial_D12.5mm_P5.00mm, F.Cu at (18.0, 80.0)
- added C4: 1000uF_25V, Capacitor_THT:CP_Radial_D12.5mm_P5.00mm, F.Cu at (18.0, 93.0)
- added C5: 1000uF_25V, Capacitor_THT:CP_Radial_D12.5mm_P5.00mm, F.Cu at (92.0, 28.0)
- added C6: 470uF_25V, Capacitor_THT:CP_Radial_D10.0mm_P5.00mm, F.Cu at (92.0, 44.0)
- added FB1: FB_DNP, Inductor_SMD:L_0603_1608Metric, F.Cu at (102.0, 13.0)
- added H1: MountingHole_M3, MountingHole:MountingHole_3.2mm_M3, F.Cu at (14.0, 14.0)
- added H2: MountingHole_M3, MountingHole:MountingHole_3.2mm_M3, F.Cu at (118.0, 14.0)
- added H3: MountingHole_M3, MountingHole:MountingHole_3.2mm_M3, F.Cu at (14.0, 96.0)
- added H4: MountingHole_M3, MountingHole:MountingHole_3.2mm_M3, F.Cu at (118.0, 96.0)
- added J1: XT60_4S_IN, Connector_AMASS:AMASS_XT60-M_1x02_P7.20mm_Vertical, F.Cu at (19.0, 24.0)
- added J10: SSD1331_OLED, Connector_PinHeader_2.54mm:PinHeader_1x07_P2.54mm_Vertical, F.Cu at (95.0, 92.0)
- added J11: WS2812B_Strip, Connector_JST:JST_XH_B3B-XH-A_1x03_P2.50mm_Vertical, F.Cu at (114.0, 92.0)
- added J12: XT30_JET_12V, Connector_AMASS:AMASS_XT30U-M_1x02_P5.0mm_Vertical, F.Cu at (114.0, 70.0)
- added J13: XT30_L2_12V, Connector_AMASS:AMASS_XT30U-M_1x02_P5.0mm_Vertical, F.Cu at (114.0, 80.0)
- added J2: UBEC_5V_AUX, Connector_PinHeader_2.54mm:PinHeader_1x03_P2.54mm_Vertical, F.Cu at (14.0, 62.0)
- added J3: XT30_Inj, Connector_AMASS:AMASS_XT30U-M_1x02_P5.0mm_Vertical, F.Cu at (114.0, 20.0)
- added J4: XT30_Inj, Connector_AMASS:AMASS_XT30U-M_1x02_P5.0mm_Vertical, F.Cu at (114.0, 30.0)
- added J5: XT30_Inj, Connector_AMASS:AMASS_XT30U-M_1x02_P5.0mm_Vertical, F.Cu at (114.0, 40.0)
- added J6: XT30_Inj, Connector_AMASS:AMASS_XT30U-M_1x02_P5.0mm_Vertical, F.Cu at (114.0, 50.0)
- added J7: XT30_Inj, Connector_AMASS:AMASS_XT30U-M_1x02_P5.0mm_Vertical, F.Cu at (114.0, 60.0)
- added J8: ServoBus_TTL, Connector_JST:JST_XH_B3B-XH-A_1x03_P2.50mm_Vertical, F.Cu at (110.0, 13.0)
- added J9: FE-URT-1, Connector_PinHeader_2.54mm:PinHeader_1x02_P2.54mm_Vertical, F.Cu at (30.0, 58.0)
- added JP1: JP_BUS_MASTER, Connector_PinHeader_2.54mm:PinHeader_1x03_P2.54mm_Vertical, F.Cu at (27.0, 66.0)
- added L1: 22uH, Inductor_SMD:L_12x12mm_H8mm, F.Cu at (92.0, 60.0)
- added M1: Voltmeter_DC, Connector_PinHeader_2.54mm:PinHeader_1x02_P2.54mm_Vertical, F.Cu at (14.0, 50.0)
- added Q1: IRLB3034PBF, Package_TO_SOT_THT:TO-220-3_Vertical, F.Cu at (34.0, 24.0)
- added Q2: BSS138_cutoff, Package_TO_SOT_SMD:SOT-23, F.Cu at (40.0, 40.0)
- added R1: 22R_DNP, Resistor_SMD:R_0603_1608Metric, F.Cu at (98.0, 13.0)
- added R10: DNP_tune, Resistor_SMD:R_0603_1608Metric, F.Cu at (36.0, 34.0)
- added R11: DNP_tune, Resistor_SMD:R_0603_1608Metric, F.Cu at (74.0, 40.0)
- added R12: DNP_tune, Resistor_SMD:R_0603_1608Metric, F.Cu at (74.0, 44.0)
- added R2: DNP_tune, Resistor_SMD:R_0603_1608Metric, F.Cu at (44.0, 40.0)
- added R3: DNP_tune, Resistor_SMD:R_0603_1608Metric, F.Cu at (48.0, 40.0)
- added R4: DNP_tune, Resistor_SMD:R_0603_1608Metric, F.Cu at (44.0, 36.0)
- added R5: DNP_tune, Resistor_SMD:R_0603_1608Metric, F.Cu at (48.0, 36.0)
- added R6: DNP_tune, Resistor_SMD:R_0603_1608Metric, F.Cu at (44.0, 32.0)
- added R7: DNP_tune, Resistor_SMD:R_0603_1608Metric, F.Cu at (48.0, 32.0)
- added R8: DNP_tune, Resistor_SMD:R_0603_1608Metric, F.Cu at (44.0, 44.0)
- added R9: DNP_tune, Resistor_SMD:R_0603_1608Metric, F.Cu at (44.0, 28.0)
- added SW1: Rocker_30A, TerminalBlock_Philmore:TerminalBlock_Philmore_TB132_1x02_P5.00mm_Horizontal, F.Cu at (19.0, 36.0)
- added SW2: Estop_NC_latching, TerminalBlock_Philmore:TerminalBlock_Philmore_TB132_1x02_P5.00mm_Horizontal, F.Cu at (26.0, 94.0)
- added U1: Pololu_D42V110F7_LEG_7V5, nova_v6:Pololu_D42V110Fx, F.Cu at (38.0, 36.0)
- added U10: INA226, nova_v6:INA226_Module_Breakout, F.Cu at (90.0, 52.0)
- added U11: INA226, nova_v6:INA226_Module_Breakout, F.Cu at (90.0, 78.0)
- added U12: Arduino_Nano_v3.x, Module:Arduino_Nano, F.Cu at (77.5, 95.5)
- added U2: Pololu_D42V110F12_HIP_12V, nova_v6:Pololu_D42V110Fx, F.Cu at (38.0, 78.0)
- added U3: Pololu_D24V22F12_L2_12V, nova_v6:Pololu_D24V22Fx, F.Cu at (62.0, 90.0)
- added U4: Pololu_D42V55F12_JET_12V, nova_v6:Pololu_D42V55Fx, F.Cu at (66.0, 30.0)
- added U5: Pololu_D42V55F7_ARM_7V5, nova_v6:Pololu_D42V55Fx, F.Cu at (66.0, 62.0)
- added U6: Teensy4.1, nova_v6:Teensy_4.1, F.Cu at (60.0, 48.0)
- added U7: 74HC125, Package_SO:SOIC-14_3.9x8.7mm_P1.27mm, F.Cu at (40.0, 65.0)
- added U8: LM393, Package_SO:SOIC-8_3.9x4.9mm_P1.27mm, F.Cu at (40.0, 52.0)
- added U9: INA226, nova_v6:INA226_Module_Breakout, F.Cu at (90.0, 26.0)
Other:
- board outline added: 112 x 90 mm
