File: hardware/pcb-mods/nova_pcb_v6_power/02_power_rails.kicad_sch (KiCad schematic)
At the start: 10 parts, among them J12 XT30_JET_12V, J13 XT30_L2_12V, J2 UBEC_5V_AUX, U1 Pololu_D42V110F7_LEG_7V5, U2 Pololu_D42V110F12_HIP_12V, U3 Pololu_D24V22F12_L2_12V, U4 Pololu_D42V55F12_JET_12V, U5 Pololu_D42V55F7_ARM_7V5

Commit message: pcb(v6-power-v2): fork to v2 — full reroute, safety chain, off-board INA226, DRC clean
- Fork nova_pcb_v6_power -> _v2 (v1 frozen); placement redone power-flow-first
- Safety chain board sync: Q3 e-stop inverter, Q4 EN_JET cutoff, R16, C8/C9
- INA226 modules converted off-board: footprints stripped to 4-pin I2C headers,
  RAW nets eliminated (bench wiring card in ROUTING_HANDOFF.md Step 8)
- All power routed 1.5/3.0mm per netclass, LEG pour L-shape, hip doubled F+B
- All signal nets routed headless via pre-commit collision checker:
  B.Cu lanes y137.5-139.9 + F.Cu verticals + via pairs; V5_AUX spine gap
  bridged x114.5; board min via relaxed to 0.45/0.25 (PCBWay standard)
- DRC: 0 errors, 0 unrouted; 2 zone-island seams left for GUI (Step 9)

Co-Authored-By: Claude Fable 5 <noreply@anthropic.com>
Parts:
- added C8, C9: 470uF_25V, Capacitor_THT:CP_Radial_D10.0mm_P5.00mm, symbol Device:C
Connections:
- net GND: now also C8.2, C9.2
- net VBAT_PROTECTED: now also C8.1, C9.1; no longer U4.3 (Pin_3)
- new net EN_JET: U4.3 (Pin_3)
