File: hardware/pcb-mods/nova_pcb_v6_power/06_safety_chain.kicad_sch (KiCad schematic)
At the start: 17 parts, among them Q2 BSS138_cutoff, SW2 Estop_NC_latching, U10 INA226, U11 INA226, U8 LM393, U9 INA226

Commit message: pcb(v6-power-v2): fork to v2 — full reroute, safety chain, off-board INA226, DRC clean
- Fork nova_pcb_v6_power -> _v2 (v1 frozen); placement redone power-flow-first
- Safety chain board sync: Q3 e-stop inverter, Q4 EN_JET cutoff, R16, C8/C9
- INA226 modules converted off-board: footprints stripped to 4-pin I2C headers,
  RAW nets eliminated (bench wiring card in ROUTING_HANDOFF.md Step 8)
- All power routed 1.5/3.0mm per netclass, LEG pour L-shape, hip doubled F+B
- All signal nets routed headless via pre-commit collision checker:
  B.Cu lanes y137.5-139.9 + F.Cu verticals + via pairs; V5_AUX spine gap
  bridged x114.5; board min via relaxed to 0.45/0.25 (PCBWay standard)
- DRC: 0 errors, 0 unrouted; 2 zone-island seams left for GUI (Step 9)

Co-Authored-By: Claude Fable 5 <noreply@anthropic.com>
Parts:
- removed R10: DNP_tune, Resistor_SMD:R_0603_1608Metric, symbol Device:R
- added C7: 100nF, Capacitor_SMD:C_0603_1608Metric, symbol Device:C
- added Q3: BSS138_estop, Package_TO_SOT_SMD:SOT-23, symbol Transistor_FET:Q_NMOS_GSD
- added Q4: BSS138_jetcut, Package_TO_SOT_SMD:SOT-23, symbol Transistor_FET:Q_NMOS_GSD
- added R13: 10k, Resistor_SMD:R_0603_1608Metric, symbol Device:R
- added R14: 470k, Resistor_SMD:R_0603_1608Metric, symbol Device:R
- added R15: 1M, Resistor_SMD:R_0603_1608Metric, symbol Device:R
- added R16: 100k, Resistor_SMD:R_0603_1608Metric, symbol Device:R
- R11, R12: value DNP_tune -> 4.7k; now fitted
- R2: value DNP_tune -> 100k; now fitted
- R3: value DNP_tune -> 22k; now fitted
- R4: value DNP_tune -> 11.3k; now fitted
- R5, R7, R8, R9: value DNP_tune -> 10k; now fitted
- R6: value DNP_tune -> 12.1k; now fitted
Connections:
- net BATT_LOW: now also R15.1
- net EN_BUCKS: now also Q3.3 (D); no longer SW2.2 (B)
- net GND: now also SW2.1 (A), C7.2, Q3.2 (S), Q4.2 (S), R16.2
- net HARDCUT: now also Q4.1 (G), R14.1, R16.1
- net V5_AUX: now also R13.2; no longer SW2.1 (A)
- net VREF_G: now also R15.2
- net VREF_H: now also R14.2
- net VSENSE: now also C7.1
- new net EN_JET: Q4.3 (D)
- new net EN_SW: Q3.1 (G), R13.1, SW2.2 (B)
