File: hardware/pcb-mods/nova_pcb_v6_logic/nova_pcb_v6_logic.kicad_sch (KiCad schematic)
At the start: 0 parts

Commit message: fix(logic): +3V3 sourced from Teensy 3.3V (T3V3O pin added) — board-killer bug fixed
Netlist verified: +3V3 = [U6.T3V3O(3V3), U7.10/13/14(VCC), J20.5]. 74HC125
+ 3x INA226 now powered. Combined with R1/FB1 un-DNP, both logic-board
bugs from the 2026-06-13 review are resolved. Board left unrouted-clean
for autorouting (Freerouting).

Co-Authored-By: Claude Fable 5 <noreply@anthropic.com>
Changed lines of the file:
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@@
 	(paper "A4")
 	(sheet
+		(at 38.1 76.2)
+		(size 88.9 25.4)
+		(exclude_from_sim no)
+		(in_bom yes)
+		(on_board yes)
+		(dnp no)
+		(fields_autoplaced yes)
+		(stroke
+			(width 0.1524)
+			(type solid)
+		)
+		(fill
+			(color 0 0 0 0.0000)
+		)
+		(property "Sheetname" "07 Aux MCU + Peripherals"
+			(at 38.1 75.4884 0)
+			(effects
+				(font
+					(size 1.27 1.27)
+				)
+				(justify left bottom)
+			)
+		)
+		(property "Sheetfile" "07_aux_mcu.kicad_sch"
+			(at 38.1 102.1772 0)
+			(effects
+				(font
+					(size 1.27 1.27)
+				)
+				(justify left top)
+			)
+		)
+		(instances
+			(project "nova_pcb_v6_logic"
+				(path "/f535083b-f621-4317-a378-cf746e7f972b"
+					(page "4")
+				)
+			)
+		)
+	)
+	(sheet
+		(at 152.4 38.1)
+		(size 88.9 25.4)
+		(exclude_from_sim no)
+		(in_bom yes)
+		(on_board yes)
+		(dnp no)
+		(fields_autoplaced yes)
+		(stroke
+			(width 0.1524)
+			(type solid)
+		)
+		(fill
+			(color 0 0 0 0.0000)
+		)
+		(property "Sheetname" "05 Bus Integrity"
+			(at 152.4 37.3884 0)
+			(effects
+				(font
+					(size 1.27 1.27)
+				)
+				(justify left bottom)
+			)
+		)
+		(property "Sheetfile" "05_bus_integrity.kicad_sch"
+			(at 152.4 64.0772 0)
+			(effects
+				(font
+					(size 1.27 1.27)
+				)
+				(justify left top)
+			)
+		)
+		(instances
+			(project "nova_pcb_v6_logic"
+				(path "/f535083b-f621-4317-a378-cf746e7f972b"
+					(page "3")
+				)
+			)
+		)
+	)
+	(sheet
+		(at 38.1 114.3)
+		(size 88.9 25.4)
+		(exclude_from_sim no)
+		(in_bom yes)
+		(on_board yes)
+		(dnp no)
+		(fields_autoplaced yes)
+		(stroke
+			(width 0.1524)
+			(type solid)
+		)
+		(fill
+			(color 0 0 0 0.0000)
+		)
+		(property "Sheetname" "09 Inter-Board Connector"
+			(at 38.1 113.5884 0)
+			(effects
+				(font
+					(size 1.27 1.27)
+				)
+				(justify left bottom)
+			)
+		)
+		(property "Sheetfile" "09_interboard.kicad_sch"
+			(at 38.1 140.2772 0)
+			(effects
+				(font
+					(size 1.27 1.27)
+				)
+				(justify left top)
+			)
+		)
+		(instances
+			(project "nova_pcb_v6_logic"
+				(path "/f535083b-f621-4317-a378-cf746e7f972b"
+					(page "6")
+				)
+			)
+		)
+	)
+	(sheet
+		(at 152.4 76.2)
+		(size 88.9 25.4)
+		(exclude_from_sim no)
+		(in_bom yes)
+		(on_board yes)
+		(dnp no)
+		(fields_autoplaced yes)
+		(stroke
+			(width 0.1524)
+			(type solid)
+		)
+		(fill
+			(color 0 0 0 0.0000)
+		)
+		(property "Sheetname" "08 Connectors + Mechanical"
+			(at 152.4 75.4884 0)
+			(effects
+				(font
+					(size 1.27 1.27)
+				)
+				(justify left bottom)
+			)
+		)
+		(property "Sheetfile" "08_connectors.kicad_sch"
+			(at 152.4 102.1772 0)
+			(effects
+				(font
+					(size 1.27 1.27)
+				)
+				(justify left top)
+			)
+		)
+		(instances
+			(project "nova_pcb_v6_logic"
+				(path "/f535083b-f621-4317-a378-cf746e7f972b"
+					(page "5")
+				)
+			)
+		)
+	)
+	(sheet
 		(at 38.1 38.1)
 		(size 88.9 25.4)
+		(exclude_from_sim no)
+		(in_bom yes)
+		(on_board yes)
+		(dnp no)
 		(fields_autoplaced yes)
 		(stroke
@@
 				(path "/f535083b-f621-4317-a378-cf746e7f972b"
 					(page "2")
-				)
-			)
-		)
-	)
-	(sheet
-		(at 152.4 38.1)
-		(size 88.9 25.4)
-		(fields_autoplaced yes)
-		(stroke
-			(width 0.1524)
-			(type solid)
-		)
-		(fill
-			(color 0 0 0 0.0000)
-		)
-		(property "Sheetname" "05 Bus Integrity"
-			(at 152.4 37.3884 0)
-			(effects
-				(font
-					(size 1.27 1.27)
-				)
-				(justify left bottom)
-			)
-		)
-		(property "Sheetfile" "05_bus_integrity.kicad_sch"
-			(at 152.4 64.0772 0)
-			(effects
-				(font
-					(size 1.27 1.27)
-				)
-				(justify left top)
-			)
-		)
-		(instances
-			(project "nova_pcb_v6_logic"
-				(path "/f535083b-f621-4317-a378-cf746e7f972b"
-					(page "3")
-				)
-			)
-		)
-	)
-	(sheet
-		(at 38.1 76.2)
-		(size 88.9 25.4)
-		(fields_autoplaced yes)
-		(stroke
-			(width 0.1524)
-			(type solid)
-		)
-		(fill
-			(color 0 0 0 0.0000)
-		)
-		(property "Sheetname" "07 Aux MCU + Peripherals"
-			(at 38.1 75.4884 0)
-			(effects
-				(font
-					(size 1.27 1.27)
-				)
-				(justify left bottom)
-			)
-		)
-		(property "Sheetfile" "07_aux_mcu.kicad_sch"
-			(at 38.1 102.1772 0)
-			(effects
-				(font
-					(size 1.27 1.27)
-				)
-				(justify left top)
-			)
-		)
-		(instances
-			(project "nova_pcb_v6_logic"
-				(path "/f535083b-f621-4317-a378-cf746e7f972b"
-					(page "4")
-				)
-			)
-		)
-	)
-	(sheet
-		(at 152.4 76.2)
-		(size 88.9 25.4)
-		(fields_autoplaced yes)
-		(stroke
-			(width 0.1524)
-			(type solid)
-		)
-		(fill
-			(color 0 0 0 0.0000)
-		)
-		(property "Sheetname" "08 Connectors + Mechanical"
-			(at 152.4 75.4884 0)
-			(effects
-				(font
-					(size 1.27 1.27)
-				)
-				(justify left bottom)
-			)
-		)
-		(property "Sheetfile" "08_connectors.kicad_sch"
-			(at 152.4 102.1772 0)
-			(effects
-				(font
-					(size 1.27 1.27)
-				)
-				(justify left top)
-			)
-		)
-		(instances
-			(project "nova_pcb_v6_logic"
-				(path "/f535083b-f621-4317-a378-cf746e7f972b"
-					(page "5")
-				)
-			)
-		)
-	)
-	(sheet
-		(at 38.1 114.30000000000001)
-		(size 88.9 25.4)
-		(fields_autoplaced yes)
-		(stroke
-			(width 0.1524)
-			(type solid)
-		)
-		(fill
-			(color 0 0 0 0.0000)
-		)
-		(property "Sheetname" "09 Inter-Board Connector"
-			(at 38.1 113.5884 0)
-			(effects
-				(font
-					(size 1.27 1.27)
-				)
-				(justify left bottom)
-			)
-		)
-		(property "Sheetfile" "09_interboard.kicad_sch"
-			(at 38.1 140.2772 0)
-			(effects
-				(font
-					(size 1.27 1.27)
-				)
-				(justify left top)
-			)
-		)
-		(instances
-			(project "nova_pcb_v6_logic"
-				(path "/f535083b-f621-4317-a378-cf746e7f972b"
-					(page "6")
 				)
 			)
@@
 			(page "1")
 		)
-		(path "/e76e40d6-be2f-49cd-bcdb-1dc94bab9b30"
-			(page "2")
-		)
-		(path "/45d7d740-e2f4-40d0-8d10-022e9099f66d"
-			(page "3")
-		)
-		(path "/0af7f1f2-3a0a-4436-aaa7-f191048b3c83"
-			(page "4")
-		)
-		(path "/6edc1b8a-dc4c-428d-8457-a29d39eb3953"
-			(page "5")
-		)
-		(path "/495b5e2f-8422-4126-a962-b63ae9783ab4"
-			(page "6")
-		)
-	)
+	)
