File: hardware/pcb-mods/nova_pcb_v6_logic/09_interboard.kicad_sch (KiCad schematic)
At the start: 1 part, among them J20 IB_2x06

Commit message: logic board: clear ERC (no_connects, drop unused NANO_3V3 + redundant V5_AUX PWR_FLAG)
ERC 18 errors -> 0 (2 cosmetic lib_symbol_mismatch warnings remain, board=truth).

- 07_aux_mcu: add no_connect on 16 unused Arduino Nano GPIO + pin 17 (3V3).
  Remove the floating NANO_3V3 label + its stub wire: the Nano's 3V3 output
  drives nothing (verified - OLED runs on V5_AUX/5V, +3V3 is Teensy-sourced).
- 09_interboard: remove redundant #FLG20 PWR_FLAG on V5_AUX (conflicted with
  the Nano +5V power-output pin -> pin_to_pin) + its orphaned V5_AUX label.

Board copper unchanged (schematic annotations only). The committed .kicad_pcb
was already clean (1x R7); the duplicate-R7 + 11 DRC violations existed only in
the uncommitted working tree and have been reverted. Gerbers refreshed from the
clean board.

Co-Authored-By: Claude Opus 4.8 <noreply@anthropic.com>
Changed lines of the file:
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@@
-		)
-	)
-	(global_label "V5_AUX"
-		(shape bidirectional)
-		(at 180.34 120.65 0)
-		(effects
-			(font
-				(size 1.27 1.27)
-			)
-			(justify left)
-		)
-		(property "Intersheetrefs" "${INTERSHEET_REFS}"
-			(at 180.34 120.65 0)
-			(effects
-				(font
-					(size 1.27 1.27)
-				)
-				(hide yes)
-			)
 		)
 	)
@@
 			)
 		)
-	)
-	(symbol
-		(lib_id "power:PWR_FLAG")
-		(at 180.34 120.65 0)
-		(unit 1)
-		(exclude_from_sim no)
-		(in_bom yes)
-		(on_board yes)
-		(dnp no)
-		(property "Reference" "#FLG20"
-			(at 180.34 114.3 0)
-			(effects
-				(font
-					(size 1.27 1.27)
-				)
-				(hide yes)
-			)
-		)
-		(property "Value" "PWR_FLAG"
-			(at 180.34 127 0)
-			(effects
-				(font
-					(size 1.27 1.27)
-				)
-				(hide yes)
-			)
-		)
-		(property "Footprint" ""
-			(at 180.34 120.65 0)
-			(effects
-				(font
-					(size 1.27 1.27)
-				)
-				(hide yes)
-			)
-		)
-		(property "Datasheet" "~"
-			(at 180.34 120.65 0)
-			(effects
-				(font
-					(size 1.27 1.27)
-				)
-				(hide yes)
-			)
-		)
-		(property "Description" ""
-			(at 180.34 120.65 0)
-			(effects
-				(font
-					(size 1.27 1.27)
-				)
-			)
-		)
-		(pin "1"
-		)
-		(instances
-			(project "nova_pcb_v6_logic"
-				(path "/f535083b-f621-4317-a378-cf746e7f972b/495b5e2f-8422-4126-a962-b63ae9783ab4"
-					(reference "#FLG20")
-					(unit 1)
-				)
-			)
-		)
