File: hardware/pcb-mods/nova_pcb_v6_logic/nova_pcb_v6_logic.kicad_pcb (KiCad board)
At the start: 4 copper layers, 84 x 78 mm, 21 parts, among them J10 SSD1331_OLED, J11 WS2812B_Strip, J20 IB_2x06, J21 Conn_01x02, J9 FE-URT-1, U12 Arduino_Nano_v3.x, U6 Teensy4.1, U7 74HC125

Commit message: logic board: U7 -> SN74LVC125A (5V-tolerant) + R7 bus idle pull-up
Full-review findings from the servo-bus level analysis:

U7: 74HC125 -> SN74LVC125A. The 74HC125 at +3V3 is NOT 5V-tolerant
(input abs-max VCC+0.5=3.8V); the STS3215 bus is 5V-TTL, so the servo's
response would over-drive gate2's input (clamp current ~54mA through R1's
22ohm). LVC125A is a drop-in SOIC-14, VCC 3.3V (max 3.6V), 5V-tolerant
inputs, 3.3V outputs (Teensy-safe) -> correct whether bus is 3.3V or 5V.
Value-only change (was stale "74LS125" in sch / "74HC125" in pcb; both
wrong for a 3.3V rail), no reroute. Unified all 5 U7 units + pcb value.

R7 = 10k bus idle pull-up (BUS_SIGNAL -> +3V3). Half-duplex push-pull bus
floats in TX/RX turnaround; R7 holds idle HIGH. Added incrementally
(footprint + 2 hand-routed nets) without disturbing the 154 existing
tracks/pours. Routed pad1->U7.10 (+3V3), pad2 down-and-around below U7 to
the BUS_SIGNAL run (staying clear of the MASTER_A diagonal).

Both boards DRC 0/0. Logic ERC = same known items (no new). Gerbers re-cut.
BOM: order SN74LVC125AD + 10k 0603. Firmware unchanged (hardware-only).

Co-Authored-By: Claude Opus 4.8 <noreply@anthropic.com>
Parts:
- added R7: 10k, R_0603_1608Metric, F.Cu at (168.0, 72.0)
- U7: value 74HC125 -> 74LVC125
Routing:
- net BUS_SIGNAL: track 29.6 -> 40.8 mm
- net +3V3: track 111.9 -> 114.7 mm
Changed lines of the file:
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@@
 		)
 	)
+	(footprint "R_0603_1608Metric"
+		(layer "F.Cu")
+		(at 168 72)
+		(descr "Resistor SMD 0603 (1608 Metric), square (rectangular) end terminal, IPC-7351 nominal, (Body size source: IPC-SM-782 page 72, https://www.pcb-3d.com/wordpress/wp-content/uploads/ipc-sm-782a_amendment_1_and_2.pdf), generated with kicad-footprint-generator")
+		(tags "resistor")
+		(property "Reference" "R7"
+			(at 0 -1.43 0)
+			(layer "F.SilkS")
+			(effects
+				(font
+					(size 1 1)
+					(thickness 0.15)
+				)
+			)
+		)
+		(property "Value" "10k"
+			(at 0 1.43 0)
+			(layer "F.Fab")
+			(effects
+				(font
+					(size 1 1)
+					(thickness 0.15)
+				)
+			)
+		)
+		(property "Datasheet" ""
+			(at 0 0 0)
+			(layer "F.Fab")
+			(hide yes)
+			(effects
+				(font
+					(size 1.27 1.27)
+					(thickness 0.15)
+				)
+			)
+		)
+		(property "Description" ""
+			(at 0 0 0)
+			(layer "F.Fab")
+			(hide yes)
+			(effects
+				(font
+					(size 1.27 1.27)
+					(thickness 0.15)
+				)
+			)
+		)
+		(attr smd)
+		(fp_line
+			(start -0.237258 -0.5225)
+			(end 0.237258 -0.5225)
+			(stroke
+				(width 0.12)
+				(type solid)
+			)
+			(layer "F.SilkS")
+		)
+		(fp_line
+			(start -0.237258 0.5225)
+			(end 0.237258 0.5225)
+			(stroke
+				(width 0.12)
+				(type solid)
+			)
+			(layer "F.SilkS")
+		)
+		(fp_line
+			(start -1.48 -0.73)
+			(end 1.48 -0.73)
+			(stroke
+				(width 0.05)
+				(type solid)
+			)
+			(layer "F.CrtYd")
+		)
+		(fp_line
+			(start -1.48 0.73)
+			(end -1.48 -0.73)
+			(stroke
+				(width 0.05)
+				(type solid)
+			)
+			(layer "F.CrtYd")
+		)
+		(fp_line
+			(start 1.48 -0.73)
+			(end 1.48 0.73)
+			(stroke
+				(width 0.05)
+				(type solid)
+			)
+			(layer "F.CrtYd")
+		)
+		(fp_line
+			(start 1.48 0.73)
+			(end -1.48 0.73)
+			(stroke
+				(width 0.05)
+				(type solid)
+			)
+			(layer "F.CrtYd")
+		)
+		(fp_line
+			(start -0.8 -0.4125)
+			(end 0.8 -0.4125)
+			(stroke
+				(width 0.1)
+				(type solid)
+			)
+			(layer "F.Fab")
+		)
+		(fp_line
+			(start -0.8 0.4125)
+			(end -0.8 -0.4125)
+			(stroke
+				(width 0.1)
+				(type solid)
+			)
+			(layer "F.Fab")
+		)
+		(fp_line
+			(start 0.8 -0.4125)
+			(end 0.8 0.4125)
+			(stroke
+				(width 0.1)
+				(type solid)
+			)
+			(layer "F.Fab")
+		)
+		(fp_line
+			(start 0.8 0.4125)
+			(end -0.8 0.4125)
+			(stroke
+				(width 0.1)
+				(type solid)
+			)
+			(layer "F.Fab")
+		)
+		(fp_text user "${REFERENCE}"
+			(at 0 0 0)
+			(layer "F.Fab")
+			(effects
+				(font
+					(size 0.4 0.4)
+					(thickness 0.06)
+				)
+			)
+		)
+		(pad "1" smd roundrect
+			(at -0.825 0)
+			(size 0.8 0.95)
+			(layers "F.Cu" "F.Mask" "F.Paste")
+			(roundrect_rratio 0.25)
+			(net 14 "+3V3")
+		)
+		(pad "2" smd roundrect
+			(at 0.825 0)
+			(size 0.8 0.95)
+			(layers "F.Cu" "F.Mask" "F.Paste")
+			(roundrect_rratio 0.25)
+			(net 17 "BUS_SIGNAL")
+		)
+		(embedded_fonts no)
+		(model "${KICAD9_3DMODEL_DIR}/Resistor_SMD.3dshapes/R_0603_1608Metric.step"
+			(offset
+				(xyz 0 0 0)
+			)
+			(scale
+				(xyz 1 1 1)
+			)
+			(rotate
+				(xyz 0 0 0)
+			)
+		)
+	)
 	(footprint "nova_v6:Teensy_4.1"
 		(layer "F.Cu")
@@
 			)
 		)
-		(property "Value" "74HC125"
+		(property "Value" "74LVC125"
 			(at 0 5.28 0)
 			(layer "F.Fab")
@@
 	)
 	(segment
+		(start 167.175 72)
+		(end 164.47 71.27)
+		(width 0.25)
+		(layer "F.Cu")
+		(net 14)
+	)
+	(segment
 		(start 164.475 71.27)
 		(end 164.0939 71.27)
@@
 	)
 	(segment
+		(start 168.825 75.5)
+		(end 161.05 75.5)
+		(width 0.25)
+		(layer "F.Cu")
+		(net 17)
+	)
+	(segment
 		(start 166.285 88.54)
 		(end 168.825 86)
@@
 		(layer "F.Cu")
 		(net 17)
+	)
+	(segment
+		(start 168.825 72)
+		(end 168.825 75.5)
+		(width 0.25)
+		(layer "F.Cu")
+		(net 17)

Commit message: boards: fab-ready GO (both) — Q1 gate-harden + soft-start, mounting-hole keepouts, BATT_NEG zone, PWR_FLAG, fresh gerbers (separate NPTH/PTH)
Power v2: Q1 gate soft-start (R17 10k + C_gs 470nF + D1 18V zener + R_gs) on Q1_GATE,
BATT_NEG F.Cu zone (solid to Q1 source, islands merged), 7mm copper keepout all 4 holes
all layers, GND PWR_FLAG. Logic: 7mm keepout all 4 holes (V5_AUX was 0.4mm from barrel).
Both: gerbers regenerated w/ explicit layer set + separate PTH/NPTH drill (M3 holes stay
non-plated). fab_gate GO: ERC 0 / DRC 0 hard / J20 match / DNP U5+U12.

Co-Authored-By: Claude Opus 4.8 <noreply@anthropic.com>
Parts:
- R7: footprint R_0603_1608Metric -> Resistor_SMD:R_0603_1608Metric
Connections:
- U12 pad 17: /07 Aux MCU + Peripherals/NANO_3V3 -> unconnected-(U12-3V3-Pad17)
Changed lines of the file:
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@@
 	(net 3 "GND")
 	(net 4 "/04 Bus Master (Pattern B)/MASTER_A")
-	(net 5 "/07 Aux MCU + Peripherals/NANO_3V3")
+	(net 5 "unconnected-(U12-3V3-Pad17)")
 	(net 6 "/07 Aux MCU + Peripherals/OLED_CS")
 	(net 7 "/07 Aux MCU + Peripherals/SPI_MOSI")
@@
 			(drill 3.2)
 			(layers "*.Cu" "*.Mask")
+			(solder_mask_margin 0)
+			(clearance 0)
 		)
 		(embedded_fonts no)
@@
 		)
 	)
-	(footprint "R_0603_1608Metric"
+	(footprint "Resistor_SMD:R_0603_1608Metric"
 		(layer "F.Cu")
 		(at 168 72)
@@
 			)
 		)
-		(property "Datasheet" ""
+		(property "Datasheet" "~"
 			(at 0 0 0)
 			(layer "F.Fab")
@@
 			)
 		)
+		(property ki_fp_filters "R_*")
+		(sheetname "/05 Bus Integrity/")
+		(sheetfile "05_bus_integrity.kicad_sch")
 		(attr smd)
 		(fp_line
@@
 			(roundrect_rratio 0.25)
 			(net 14 "+3V3")
+			(pintype "passive")
 		)
 		(pad "2" smd roundrect
@@
 			(roundrect_rratio 0.25)
 			(net 17 "BUS_SIGNAL")
+			(pintype "passive")
 		)
 		(embedded_fonts no)
@@
 			(drill 3.2)
 			(layers "*.Cu" "*.Mask")
+			(solder_mask_margin 0)
+			(clearance 0)
 		)
 		(embedded_fonts no)
@@
 			(drill 3.2)
 			(layers "*.Cu" "*.Mask")
+			(solder_mask_margin 0)
+			(clearance 0)
 		)
 		(embedded_fonts no)
@@
 			(net 31 "unconnected-(U12-D1{slash}TX-Pad1)")
 			(pinfunction "D1/TX")
-			(pintype "bidirectional")
+			(pintype "bidirectional+no_connect")
 		)
 		(pad "2" thru_hole oval
@@
 			(net 29 "unconnected-(U12-D0{slash}RX-Pad2)")
 			(pinfunction "D0/RX")
-			(pintype "bidirectional")
+			(pintype "bidirectional+no_connect")
 		)
 		(pad "3" thru_hole oval
@@
 			(net 42 "unconnected-(U12-D2-Pad5)")
 			(pinfunction "D2")
-			(pintype "bidirectional")
+			(pintype "bidirectional+no_connect")
 		)
 		(pad "6" thru_hole oval
@@
 			(net 28 "unconnected-(U12-D3-Pad6)")
 			(pinfunction "D3")
-			(pintype "bidirectional")
+			(pintype "bidirectional+no_connect")
 		)
 		(pad "7" thru_hole oval
@@
 			(net 37 "unconnected-(U12-D4-Pad7)")
 			(pinfunction "D4")
-			(pintype "bidirectional")
+			(pintype "bidirectional+no_connect")
 		)
 		(pad "8" thru_hole oval
@@
 			(net 34 "unconnected-(U12-D5-Pad8)")
 			(pinfunction "D5")
-			(pintype "bidirectional")
+			(pintype "bidirectional+no_connect")
 		)
 		(pad "9" thru_hole oval
@@
 			(net 44 "unconnected-(U12-D7-Pad10)")
 			(pinfunction "D7")
-			(pintype "bidirectional")
+			(pintype "bidirectional+no_connect")
 		)
 		(pad "11" thru_hole oval
@@
 			(net 38 "unconnected-(U12-D12-Pad15)")
 			(pinfunction "D12")
-			(pintype "bidirectional")
+			(pintype "bidirectional+no_connect")
 		)
 		(pad "16" thru_hole oval
@@
 			(layers "*.Cu" "*.Mask")
 			(remove_unused_layers no)
-			(net 5 "/07 Aux MCU + Peripherals/NANO_3V3")
+			(net 5 "unconnected-(U12-3V3-Pad17)")
 			(pinfunction "3V3")
-			(pintype "power_out")
+			(pintype "power_out+no_connect")
 		)
 		(pad "18" thru_hole oval
@@
 			(net 27 "unconnected-(U12-A0-Pad19)")
 			(pinfunction "A0")
-			(pintype "bidirectional")
+			(pintype "bidirectional+no_connect")
 		)
 		(pad "20" thru_hole oval
@@
 			(net 33 "unconnected-(U12-A1-Pad20)")
 			(pinfunction "A1")
-			(pintype "bidirectional")
+			(pintype "bidirectional+no_connect")
 		)
 		(pad "21" thru_hole oval
@@
 			(net 41 "unconnected-(U12-A2-Pad21)")
 			(pinfunction "A2")
-			(pintype "bidirectional")
+			(pintype "bidirectional+no_connect")
 		)
 		(pad "22" thru_hole oval
@@
 			(net 43 "unconnected-(U12-A3-Pad22)")
 			(pinfunction "A3")
-			(pintype "bidirectional")
+			(pintype "bidirectional+no_connect")
 		)
 		(pad "23" thru_hole oval
@@
 			(net 36 "unconnected-(U12-A4-Pad23)")
 			(pinfunction "A4")
-			(pintype "bidirectional")
+			(pintype "bidirectional+no_connect")
 		)
 		(pad "24" thru_hole oval
@@
 			(net 32 "unconnected-(U12-A5-Pad24)")
 			(pinfunction "A5")
-			(pintype "bidirectional")
+			(pintype "bidirectional+no_connect")
 		)
 		(pad "25" thru_hole oval
@@
 			(net 40 "unconnected-(U12-A6-Pad25)")
 			(pinfunction "A6")
-			(pintype "bidirectional")
+			(pintype "bidirectional+no_connect")
 		)
 		(pad "26" thru_hole oval
@@
 			(net 30 "unconnected-(U12-A7-Pad26)")
 			(pinfunction "A7")
-			(pintype "bidirectional")
+			(pintype "bidirectional+no_connect")
 		)
 		(pad "27" thru_hole oval
@@
 			(drill 3.2)
 			(layers "*.Cu" "*.Mask")
+			(solder_mask_margin 0)
+			(clearance 0)
 		)
 		(embedded_fonts no)
@@
 			)
 		)
+	)
+	(zone
+		(net 0)
+		(net_name "")
+		(layers "F.Cu" "B.Cu" "In1.Cu" "In2.Cu")
+		(hatch edge 0.5)
+		(connect_pads
+			(clearance 0)
+		)
+		(min_thickness 0.25)
+		(filled_areas_thickness no)
+		(keepout
+			(tracks allowed)
+			(vias allowed)
+			(pads allowed)
+			(copperpour not_allowed)
+			(footprints allowed)
+		)
+		(placement
+			(enabled no)
+			(sheetname "")
+		)
+		(fill
+			(thermal_gap 0.5)
+			(thermal_bridge_width 0.5)
+		)
+		(polygon
+			(pts
+				(xy 106.5 129) (xy 106.432748 129.682816) (xy 106.233578 130.339392) (xy 105.910143 130.944495)
+				(xy 105.474873 131.474873) (xy 104.944495 131.910143) (xy 104.339392 132.233578) (xy 103.682816 132.432748)
+				(xy 103 132.5) (xy 102.317183 132.432748) (xy 101.660607 132.233578) (xy 101.055504 131.910143)
+				(xy 100.525126 131.474873) (xy 100.089856 130.944495) (xy 99.766421 130.339392) (xy 99.567251 129.682816)
+				(xy 99.5 129) (xy 99.567251 128.317183) (xy 99.766421 127.660607) (xy 100.089856 127.055504) (xy 100.525126 126.525126)
+				(xy 101.055504 126.089856) (xy 101.660607 125.766421) (xy 102.317183 125.567251) (xy 103 125.5)
+				(xy 103.682816 125.567251) (xy 104.339392 125.766421) (xy 104.944495 126.089856) (xy 105.474873 126.525126)
+				(xy 105.910143 127.055504) (xy 106.233578 127.660607) (xy 106.432748 128.317183)
+			)
+		)
+	)
+	(zone
+		(net 0)
+		(net_name "")
+		(layers "F.Cu" "B.Cu" "In1.Cu" "In2.Cu")
+		(hatch edge 0.5)
+		(connect_pads
+			(clearance 0)
+		)
+		(min_thickness 0.25)
+		(filled_areas_thickness no)
+		(keepout
+			(tracks allowed)
+			(vias allowed)
+			(pads allowed)
+			(copperpour not_allowed)
+			(footprints allowed)
+		)
+		(placement
+			(enabled no)
+			(sheetname "")
+		)
+		(fill
+			(thermal_gap 0.5)
+			(thermal_bridge_width 0.5)
+		)
+		(polygon
+			(pts
+				(xy 180.5 63) (xy 180.432748 63.682816) (xy 180.233578 64.339392) (xy 179.910143 64.944495) (xy 179.474873 65.474873)
+				(xy 178.944495 65.910143) (xy 178.339392 66.233578) (xy 177.682816 66.432748) (xy 177 66.5) (xy 176.317183 66.432748)
+				(xy 175.660607 66.233578) (xy 175.055504 65.910143) (xy 174.525126 65.474873) (xy 174.089856 64.944495)
+				(xy 173.766421 64.339392) (xy 173.567251 63.682816) (xy 173.5 63) (xy 173.567251 62.317183) (xy 173.766421 61.660607)
+				(xy 174.089856 61.055504) (xy 174.525126 60.525126) (xy 175.055504 60.089856) (xy 175.660607 59.766421)
+				(xy 176.317183 59.567251) (xy 177 59.5) (xy 177.682816 59.567251) (xy 178.339392 59.766421) (xy 178.944495 60.089856)
+				(xy 179.474873 60.525126) (xy 179.910143 61.055504) (xy 180.233578 61.660607) (xy 180.432748 62.317183)
+			)
+		)
+	)
+	(zone
+		(net 0)
+		(net_name "")
+		(layers "F.Cu" "B.Cu" "In1.Cu" "In2.Cu")
+		(hatch edge 0.5)
+		(connect_pads
+			(clearance 0)
+		)
+		(min_thickness 0.25)
+		(filled_areas_thickness no)
+		(keepout
+			(tracks allowed)
+			(vias allowed)
+			(pads allowed)
+			(copperpour not_allowed)
+			(footprints allowed)
+		)
+		(placement
+			(enabled no)
+			(sheetname "")
+		)
+		(fill
+			(thermal_gap 0.5)
+			(thermal_bridge_width 0.5)
+		)
+		(polygon
+			(pts
+				(xy 106.5 63) (xy 106.432748 63.682816) (xy 106.233578 64.339392) (xy 105.910143 64.944495) (xy 105.474873 65.474873)
+				(xy 104.944495 65.910143) (xy 104.339392 66.233578) (xy 103.682816 66.432748) (xy 103 66.5) (xy 102.317183 66.432748)
+				(xy 101.660607 66.233578) (xy 101.055504 65.910143) (xy 100.525126 65.474873) (xy 100.089856 64.944495)
+				(xy 99.766421 64.339392) (xy 99.567251 63.682816) (xy 99.5 63) (xy 99.567251 62.317183) (xy 99.766421 61.660607)
+				(xy 100.089856 61.055504) (xy 100.525126 60.525126) (xy 101.055504 60.089856) (xy 101.660607 59.766421)
+				(xy 102.317183 59.567251) (xy 103 59.5) (xy 103.682816 59.567251) (xy 104.339392 59.766421) (xy 104.944495 60.089856)
+				(xy 105.474873 60.525126) (xy 105.910143 61.055504) (xy 106.233578 61.660607) (xy 106.432748 62.317183)
+			)
+		)
+	)
+	(zone
+		(net 0)
+		(net_name "")
+		(layers "F.Cu" "B.Cu" "In1.Cu" "In2.Cu")
+		(hatch edge 0.5)
+		(connect_pads
+			(clearance 0)
+		)
+		(min_thickness 0.25)
+		(filled_areas_thickness no)
+		(keepout
+			(tracks allowed)
+			(vias allowed)
+			(pads allowed)
+			(copperpour not_allowed)
+			(footprints allowed)
+		)
+		(placement
+			(enabled no)
+			(sheetname "")
+		)
+		(fill
+			(thermal_gap 0.5)
+			(thermal_bridge_width 0.5)
+		)
+		(polygon
+			(pts
+				(xy 180.5 129) (xy 180.432748 129.682816) (xy 180.233578 130.339392) (xy 179.910143 130.944495)
+				(xy 179.474873 131.474873) (xy 178.944495 131.910143) (xy 178.339392 132.233578) (xy 177.682816 132.432748)
+				(xy 177 132.5) (xy 176.317183 132.432748) (xy 175.660607 132.233578) (xy 175.055504 131.910143)
+				(xy 174.525126 131.474873) (xy 174.089856 130.944495) (xy 173.766421 130.339392) (xy 173.567251 129.682816)
+				(xy 173.5 129) (xy 173.567251 128.317183) (xy 173.766421 127.660607) (xy 174.089856 127.055504)
+				(xy 174.525126 126.525126) (xy 175.055504 126.089856) (xy 175.660607 125.766421) (xy 176.317183 125.567251)
+				(xy 177 125.5) (xy 177.682816 125.567251) (xy 178.339392 125.766421) (xy 178.944495 126.089856)
+				(xy 179.474873 126.525126) (xy 179.910143 127.055504) (xy 180.233578 127.660607) (xy 180.432748 128.317183)
+			)
+		)
