File: hardware/pcb-mods/nova_pcb_v6_power_v2/nova_pcb_v6_power_v2.kicad_sch (KiCad schematic)
At the start: 0 parts

Commit message: boards: fab-ready GO (both) — Q1 gate-harden + soft-start, mounting-hole keepouts, BATT_NEG zone, PWR_FLAG, fresh gerbers (separate NPTH/PTH)
Power v2: Q1 gate soft-start (R17 10k + C_gs 470nF + D1 18V zener + R_gs) on Q1_GATE,
BATT_NEG F.Cu zone (solid to Q1 source, islands merged), 7mm copper keepout all 4 holes
all layers, GND PWR_FLAG. Logic: 7mm keepout all 4 holes (V5_AUX was 0.4mm from barrel).
Both: gerbers regenerated w/ explicit layer set + separate PTH/NPTH drill (M3 holes stay
non-plated). fab_gate GO: ERC 0 / DRC 0 hard / J20 match / DNP U5+U12.

Co-Authored-By: Claude Opus 4.8 <noreply@anthropic.com>
Changed lines of the file:
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@@
 	(paper "A4")
 	(sheet
+		(at 152.4 38.1)
+		(size 88.9 25.4)
+		(exclude_from_sim no)
+		(in_bom yes)
+		(on_board yes)
+		(dnp no)
+		(fields_autoplaced yes)
+		(stroke
+			(width 0.1524)
+			(type solid)
+		)
+		(fill
+			(color 0 0 0 0.0000)
+		)
+		(property "Sheetname" "02 Power Rails (Pololu bucks)"
+			(at 152.4 37.3884 0)
+			(effects
+				(font
+					(size 1.27 1.27)
+				)
+				(justify left bottom)
+			)
+		)
+		(property "Sheetfile" "02_power_rails.kicad_sch"
+			(at 152.4 64.0772 0)
+			(effects
+				(font
+					(size 1.27 1.27)
+				)
+				(justify left top)
+			)
+		)
+		(instances
+			(project "nova_pcb_v6_power_v2"
+				(path "/f535083b-f621-4317-a378-cf746e7f972b"
+					(page "3")
+				)
+			)
+		)
+	)
+	(sheet
+		(at 152.4 76.2)
+		(size 88.9 25.4)
+		(exclude_from_sim no)
+		(in_bom yes)
+		(on_board yes)
+		(dnp no)
+		(fields_autoplaced yes)
+		(stroke
+			(width 0.1524)
+			(type solid)
+		)
+		(fill
+			(color 0 0 0 0.0000)
+		)
+		(property "Sheetname" "06 Safety Chain"
+			(at 152.4 75.4884 0)
+			(effects
+				(font
+					(size 1.27 1.27)
+				)
+				(justify left bottom)
+			)
+		)
+		(property "Sheetfile" "06_safety_chain.kicad_sch"
+			(at 152.4 102.1772 0)
+			(effects
+				(font
+					(size 1.27 1.27)
+				)
+				(justify left top)
+			)
+		)
+		(instances
+			(project "nova_pcb_v6_power_v2"
+				(path "/f535083b-f621-4317-a378-cf746e7f972b"
+					(page "5")
+				)
+			)
+		)
+	)
+	(sheet
+		(at 38.1 114.3)
+		(size 88.9 25.4)
+		(exclude_from_sim no)
+		(in_bom yes)
+		(on_board yes)
+		(dnp no)
+		(fields_autoplaced yes)
+		(stroke
+			(width 0.1524)
+			(type solid)
+		)
+		(fill
+			(color 0 0 0 0.0000)
+		)
+		(property "Sheetname" "08 Connectors + Mechanical"
+			(at 38.1 113.5884 0)
+			(effects
+				(font
+					(size 1.27 1.27)
+				)
+				(justify left bottom)
+			)
+		)
+		(property "Sheetfile" "08_connectors.kicad_sch"
+			(at 38.1 140.2772 0)
+			(effects
+				(font
+					(size 1.27 1.27)
+				)
+				(justify left top)
+			)
+		)
+		(instances
+			(project "nova_pcb_v6_power_v2"
+				(path "/f535083b-f621-4317-a378-cf746e7f972b"
+					(page "6")
+				)
+			)
+		)
+	)
+	(sheet
+		(at 38.1 76.2)
+		(size 88.9 25.4)
+		(exclude_from_sim no)
+		(in_bom yes)
+		(on_board yes)
+		(dnp no)
+		(fields_autoplaced yes)
+		(stroke
+			(width 0.1524)
+			(type solid)
+		)
+		(fill
+			(color 0 0 0 0.0000)
+		)
+		(property "Sheetname" "03 Servo Bus (star injection)"
+			(at 38.1 75.4884 0)
+			(effects
+				(font
+					(size 1.27 1.27)
+				)
+				(justify left bottom)
+			)
+		)
+		(property "Sheetfile" "03_servo_bus.kicad_sch"
+			(at 38.1 102.1772 0)
+			(effects
+				(font
+					(size 1.27 1.27)
+				)
+				(justify left top)
+			)
+		)
+		(instances
+			(project "nova_pcb_v6_power_v2"
+				(path "/f535083b-f621-4317-a378-cf746e7f972b"
+					(page "4")
+				)
+			)
+		)
+	)
+	(sheet
 		(at 38.1 38.1)
 		(size 88.9 25.4)
+		(exclude_from_sim no)
+		(in_bom yes)
+		(on_board yes)
+		(dnp no)
 		(fields_autoplaced yes)
 		(stroke
@@
 	)
 	(sheet
-		(at 152.4 38.1)
-		(size 88.9 25.4)
-		(fields_autoplaced yes)
-		(stroke
-			(width 0.1524)
-			(type solid)
-		)
-		(fill
-			(color 0 0 0 0.0000)
-		)
-		(property "Sheetname" "02 Power Rails (Pololu bucks)"
-			(at 152.4 37.3884 0)
-			(effects
-				(font
-					(size 1.27 1.27)
-				)
-				(justify left bottom)
-			)
-		)
-		(property "Sheetfile" "02_power_rails.kicad_sch"
-			(at 152.4 64.0772 0)
-			(effects
-				(font
-					(size 1.27 1.27)
-				)
-				(justify left top)
-			)
-		)
-		(instances
-			(project "nova_pcb_v6_power_v2"
-				(path "/f535083b-f621-4317-a378-cf746e7f972b"
-					(page "3")
-				)
-			)
-		)
-	)
-	(sheet
-		(at 38.1 76.2)
-		(size 88.9 25.4)
-		(fields_autoplaced yes)
-		(stroke
-			(width 0.1524)
-			(type solid)
-		)
-		(fill
-			(color 0 0 0 0.0000)
-		)
-		(property "Sheetname" "03 Servo Bus (star injection)"
-			(at 38.1 75.4884 0)
-			(effects
-				(font
-					(size 1.27 1.27)
-				)
-				(justify left bottom)
-			)
-		)
-		(property "Sheetfile" "03_servo_bus.kicad_sch"
-			(at 38.1 102.1772 0)
-			(effects
-				(font
-					(size 1.27 1.27)
-				)
-				(justify left top)
-			)
-		)
-		(instances
-			(project "nova_pcb_v6_power_v2"
-				(path "/f535083b-f621-4317-a378-cf746e7f972b"
-					(page "4")
-				)
-			)
-		)
-	)
-	(sheet
-		(at 152.4 76.2)
-		(size 88.9 25.4)
-		(fields_autoplaced yes)
-		(stroke
-			(width 0.1524)
-			(type solid)
-		)
-		(fill
-			(color 0 0 0 0.0000)
-		)
-		(property "Sheetname" "06 Safety Chain"
-			(at 152.4 75.4884 0)
-			(effects
-				(font
-					(size 1.27 1.27)
-				)
-				(justify left bottom)
-			)
-		)
-		(property "Sheetfile" "06_safety_chain.kicad_sch"
-			(at 152.4 102.1772 0)
-			(effects
-				(font
-					(size 1.27 1.27)
-				)
-				(justify left top)
-			)
-		)
-		(instances
-			(project "nova_pcb_v6_power_v2"
-				(path "/f535083b-f621-4317-a378-cf746e7f972b"
-					(page "5")
-				)
-			)
-		)
-	)
-	(sheet
-		(at 38.1 114.30000000000001)
-		(size 88.9 25.4)
-		(fields_autoplaced yes)
-		(stroke
-			(width 0.1524)
-			(type solid)
-		)
-		(fill
-			(color 0 0 0 0.0000)
-		)
-		(property "Sheetname" "08 Connectors + Mechanical"
-			(at 38.1 113.5884 0)
-			(effects
-				(font
-					(size 1.27 1.27)
-				)
-				(justify left bottom)
-			)
-		)
-		(property "Sheetfile" "08_connectors.kicad_sch"
-			(at 38.1 140.2772 0)
-			(effects
-				(font
-					(size 1.27 1.27)
-				)
-				(justify left top)
-			)
-		)
-		(instances
-			(project "nova_pcb_v6_power_v2"
-				(path "/f535083b-f621-4317-a378-cf746e7f972b"
-					(page "6")
-				)
-			)
-		)
-	)
-	(sheet
-		(at 152.4 114.30000000000001)
-		(size 88.9 25.4)
+		(at 152.4 114.3)
+		(size 88.9 25.4)
+		(exclude_from_sim no)
+		(in_bom yes)
+		(on_board yes)
+		(dnp no)
 		(fields_autoplaced yes)
 		(stroke
@@
 			(page "1")
 		)
-		(path "/ef143087-bea8-42bd-8bca-c15c2f4ac5f7"
-			(page "2")
-		)
-		(path "/27a07a1d-f9e1-432b-b0b9-19fa0d701a09"
-			(page "3")
-		)
-		(path "/8f3fe7b3-c0aa-43f7-a2b9-c8492e89dcc9"
-			(page "4")
-		)
-		(path "/38477265-f64f-4f2e-aefb-289b79c664e1"
-			(page "5")
-		)
-		(path "/6edc1b8a-dc4c-428d-8457-a29d39eb3953"
-			(page "6")
-		)
-		(path "/fa111b54-7a85-49af-8eb1-99842a09914c"
-			(page "7")
-		)
-	)
+	)
