File: hardware/pcb-mods/nova_pcb_v6_power_v2/06_safety_chain.kicad_sch (KiCad schematic)
At the start: 24 parts, among them Q2 BSS138_cutoff, Q3 BSS138_estop, Q4 BSS138_jetcut, SW2 Estop_NC_latching, U10 INA226, U11 INA226, U12 INA226, U8 LM393, U9 INA226

Commit message: power board: fix reversed XT connector polarity (all 9 AMASS XT)
AMASS XT footprints number pad1=chamfer/NEGATIVE, pad2=flat/POSITIVE.
Board had +V wired to pad1 -> every keyed power connector reverse-wired:
J1 (XT60 battery in), J3-J7 (rail injection), J12-J14 (Jetson/L2/arm out).
Mating a normally-built cable would feed +V to the - terminal and fry the
connected load (Jetson, servos, arm). Confirmed against footprint flat/chamfer
geometry + physical connector (flat=+).

Fix: swapped pin1/pin2 net assignment on all 9 connectors in schematic,
re-routed PCB, regenerated 14-file gerber set. Pololu bucks use a custom
non-keyed terminal (pad1=rect=+V) and were correctly left unchanged.

Verify: ERC 0, DRC 0 hard / 0 unconnected, fab_gate GO, J20 match intact.

Co-Authored-By: Claude Opus 4.8 <noreply@anthropic.com>
Other:
- moved on the sheet: R11, R13, U12
