File: hardware/pcb-mods/nova_pcb_v6_power_v2/02_power_rails.kicad_sch (KiCad schematic)
At the start: 13 parts, among them J12 XT30_JET_12V, J13 XT30_L2_12V, J14 XT30_Arm7V5, J2 UBEC_5V_AUX, U1 Pololu_D42V110F7_LEG_7V5, U2 Pololu_D42V110F12_HIP_12V, U3 Pololu_D24V22F12_L2_12V, U4 Pololu_D42V55F12_JET_12V, U5 Pololu_D42V55F7_ARM_7V5

Commit message: Chassis + leg_v6 CAD: no-drill assembly, leg fault audit (LA-1..28 + #47), fastener + gate hardening (#48)
* power board: arm Phase-4 routed + cleaned + fresh gerbers (fab-ready)

Completes the power board (blocker B1):
- U5.EN routed on EN_BUCKS (re-gate now realized on the board).
- V7V5_ARM 3mm, BATT_NEG/VBAT long runs 3mm, 21 high-current pads solid
  zone-connection (current-capacity fixes; TO-220/SW1 escapes left at 1.3mm).
- Removed the duplicate U12 + J14 (F8 UUID-mismatch artifacts) and the full
  orphan dangling-track chain they left behind.
- DRC: 0 hard, 0 unconnected, 0 dangling (10 cosmetic silk/lib only).
- Gerbers regenerated; fab_gate GO on both boards (J20 cross-board match OK).

DNP roster correct (U5 arm buck, U12 arm INA = Phase-4 reserve).

Co-Authored-By: Claude Opus 4.8 <noreply@anthropic.com>

* audit fixes 2026-06-18: NaN guard, pinout/battery/LVC doc sync, STATUS audit block

- main.cpp: NaN guard on commanded position (was UB (uint16_t)NaN -> 0 slam)
- teensy firmware/README.md: pinout table corrected to match main.cpp/PCB v6 (Serial1 0/1, E-stop 5, batt 4, active-LOW OE)
- power-budget.md + BOM.md: battery 4000->6000mAh (real Ovonic packs) + runtime/charge recompute
- BOM.md: bus driver order line -> SN74LVC125A (must be LVC, not 74HC125)
- STATUS.md: cross-domain audit section (open misalignments, weak points, questions)

Co-Authored-By: Claude Opus 4.8 <noreply@anthropic.com>

* docs: add servo-bus half-duplex timing bench checklist (pre-power-on §10)

Co-Authored-By: Claude Opus 4.8 <noreply@anthropic.com>

* docs: battery 4000->6000mAh sweep across secondary docs + STATUS CI-note fix

- 6000mAh 4S Ovonic (real pack) in cad-tooling, notes-qol (SoC math 5400mAh),
  order-list (bag), wiring diagram, README charger note, patterns pocket label
- dimensions.md + patterns.md: physical box/pocket dims flagged RE-MEASURE
  (6000mAh pack is larger; old 4000mAh dims kept as reference, not as truth)
- STATUS.md: corrected CI note (ros-pytest.yml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
Connections:
- net GND: now also J12.1 (Pin_1), J13.1 (Pin_1), J14.1 (Pin_1); no longer J12.2 (Pin_2), J13.2 (Pin_2), J14.2 (Pin_2)
- net V12_JET: now also J12.2 (Pin_2); no longer J12.1 (Pin_1)
- net V12_L2: now also J13.2 (Pin_2); no longer J13.1 (Pin_1)
- net V7V5_ARM: now also J14.2 (Pin_2); no longer J14.1 (Pin_1)
