Commit message: B2: measured femur/tibia link lengths from STL bores
Femur (hfe->kfe) 106.9mm, tibia (kfe->foot post) 129.0mm, via trimesh
slice-circle bore detection on the original NovaSM3 STLs (leg_v5 keeps
stock pivots). Propagated URDF + LegParams + trot comment; method and
per-bore coordinates recorded in dimensions.md §6.

Femur's 12mm in-plane kink is absorbed into hfe zero-calibration; IK
stays scalar-length. Still open: hip lateral offset d (needs assembled
hip or Onshape assembly), joint ranges, masses/inertias, body mounts.

Co-Authored-By: Claude Fable 5 <noreply@anthropic.com>
Claude-Session: https://claude.ai/code/session_013wnx3m6TJKxLuNtpieRaWF

File: ros2_ws/src/nova_description/urdf/nova.urdf.xacro (robot description, xacro)
@@ -31,8 +31,15 @@
   <xacro:property name="hip_to_upper_y" value="0.045"/>  <!-- TODO-CAD coax horn -> femur axis -->
   <xacro:property name="hip_to_upper_z" value="0.0"/>    <!-- TODO-CAD -->
-  <xacro:property name="upper_to_lower_x" value="0.0"/>  <!-- TODO-CAD -->
-  <xacro:property name="upper_to_lower_z" value="-0.11"/><!-- TODO-CAD femur length -->
-  <xacro:property name="lower_to_foot_x" value="0.0"/>   <!-- TODO-CAD -->
-  <xacro:property name="lower_to_foot_z" value="-0.13"/> <!-- TODO-CAD tibia length -->
+  <!-- MEASURED 2026-07-01 from original NovaSM3 STLs (leg_v5 keeps stock pivots).
+       Femur: hfe horn axis (49.5, z10) -> kfe bore (-56.71, z22.02) in
+       SM3_Frame_LeftFemur.stl = 106.9 mm axis-to-axis (the 12 mm in-plane kink
+       is absorbed into hfe zero-calibration; IK uses the scalar length).
+       Tibia: kfe spline (62.5, 0) -> foot post center (-66.5, 3.3) in
+       SM3_Frame_RightTibia.stl = 129.0 mm (toe tip extreme = 138.0 mm).
+       Method: trimesh slice-circle bore detection, hardware/cad/dimensions.md §leg. -->
+  <xacro:property name="upper_to_lower_x" value="0.0"/>
+  <xacro:property name="upper_to_lower_z" value="-0.1069"/><!-- MEASURED femur length -->
+  <xacro:property name="lower_to_foot_x" value="0.0"/>
+  <xacro:property name="lower_to_foot_z" value="-0.1290"/> <!-- MEASURED tibia length -->
   <!-- ===================== masses (kg) ===================== -->
   <!-- TODO-CAD: weigh / compute from CAD. STS3215 ≈ 0.06 kg each. -->

Commit message: leg_v6: tibia + coax + mirrors — full leg chain designed + verified
Tibia: KFE pocket + straight blade, Ø7 foot post at x=129.0 with post
span z -21..-40 (center -30.5 = the measured stock jog, so the stock
SM3_Foot rubber and the IK d both carry over; straight blade is stiffer
than the stock S-curve). Coax: HAA pocket (horn-first front insertion,
rear countersunk M2.5 into case threads, rear pad/heat-set = shoulder
yoke idler) + femur yoke with hfe at (11.6, -9.5) per A360 measurement,
bridge clears the full femur-disc sweep. L parts = mirror wrappers
($fn re-declared — dynamic scoping doesn't cross use<>).

URDF laterals redistributed for v6 (33.8/0/30.5, total 64.3 unchanged);
tests green. All six STLs watertight, features slice-verified.

Co-Authored-By: Claude Fable 5 <noreply@anthropic.com>
Claude-Session: https://claude.ai/code/session_013wnx3m6TJKxLuNtpieRaWF

File: ros2_ws/src/nova_description/urdf/nova.urdf.xacro (robot description, xacro)
@@ -35,8 +35,11 @@
   <xacro:property name="mount_z"     value="0.0380"/> <!-- hip row above chassis-mesh origin; ⚠ REVIEW-visual (trunk-node bbox polluted by children) -->
   <xacro:property name="hip_to_upper_x" value="0.0"/>
-  <xacro:property name="hip_to_upper_y" value="0.0246"/> <!-- MEASURED haa axis -> femur horn plane -->
+  <!-- v6 legs (leg_v6/) redistribute the SAME 64.3mm total: femur mid-plane
+       at 33.8 from haa (coax yoke), femur/tibia coplanar (0), foot post 30.5.
+       Stock-part values were 24.6 / 9.2 / 30.5. Total unchanged -> IK d valid. -->
+  <xacro:property name="hip_to_upper_y" value="0.0338"/> <!-- haa axis -> femur mid-plane (v6) -->
   <xacro:property name="hip_to_upper_z" value="-0.0095"/><!-- MEASURED hfe drop below haa -->
-  <xacro:property name="upper_to_lower_y" value="0.0092"/><!-- MEASURED hfe->kfe outboard shift -->
-  <xacro:property name="lower_to_foot_y"  value="0.0305"/><!-- MEASURED tibia S-curve outboard shift -->
+  <xacro:property name="upper_to_lower_y" value="0.0"/>  <!-- v6: femur/tibia coplanar -->
+  <xacro:property name="lower_to_foot_y"  value="0.0305"/><!-- foot post offset (v6 = stock jog) -->
   <!-- MEASURED 2026-07-01 from original NovaSM3 STLs (leg_v5 keeps stock pivots).
        Femur: hfe horn axis (49.5, z10) -> kfe bore (-56.71, z22.02) in

Commit message: leg_v6: flip toe jog INBOARD — foot lands 3.3mm from the roll axis
User's insight, confirmed by the numbers: stock's outboard jog puts the
foot 64.3mm from the haa axis = ~0.77 N.m of holding torque per hip
(26% of the 30kg servo rating) burned continuously while standing.
Jogging the toe tab inboard instead lands the foot 33.8 - 30.5 = 3.3mm
from the roll axis: near-zero static roll torque, and the wide stable
stance is still available on demand by rolling the hips out (Go1/
Cheetah-class geometry).

Swept-verified: tab+shoe orbit the knee at r>=114.7 vs femur fork
r<=15.85 (clear at any fold); inboard tab z-band never overlaps the
femur slab. Blade taper flipped top-flush so the raised web connects
(was 2 bodies). d propagated: URDF lower_to_foot_y -0.0305, IK
hip_offset 0.0033, trot stand_y — tests green.

Co-Authored-By: Claude Fable 5 <noreply@anthropic.com>
Claude-Session: https://claude.ai/code/session_013wnx3m6TJKxLuNtpieRaWF

File: ros2_ws/src/nova_description/urdf/nova.urdf.xacro (robot description, xacro)
@@ -35,11 +35,13 @@
   <xacro:property name="mount_z"     value="0.0380"/> <!-- hip row above chassis-mesh origin; ⚠ REVIEW-visual (trunk-node bbox polluted by children) -->
   <xacro:property name="hip_to_upper_x" value="0.0"/>
-  <!-- v6 legs (leg_v6/) redistribute the SAME 64.3mm total: femur mid-plane
-       at 33.8 from haa (coax yoke), femur/tibia coplanar (0), foot post 30.5.
-       Stock-part values were 24.6 / 9.2 / 30.5. Total unchanged -> IK d valid. -->
+  <!-- v6 legs (leg_v6/): femur mid-plane 33.8 from haa (coax yoke), femur/
+       tibia coplanar (0), and the toe tab jogs 30.5 INBOARD (v6 rev2 decision
+       2026-07-02 — opposite of stock) so the foot lands 3.3mm from the haa
+       roll axis: near-zero standing roll torque (stock's outboard jog cost
+       ~0.77 N·m/hip holding). Wide stance on demand via hip roll. -->
   <xacro:property name="hip_to_upper_y" value="0.0338"/> <!-- haa axis -> femur mid-plane (v6) -->
   <xacro:property name="hip_to_upper_z" value="-0.0095"/><!-- MEASURED hfe drop below haa -->
   <xacro:property name="upper_to_lower_y" value="0.0"/>  <!-- v6: femur/tibia coplanar -->
-  <xacro:property name="lower_to_foot_y"  value="0.0305"/><!-- foot post offset (v6 = stock jog) -->
+  <xacro:property name="lower_to_foot_y"  value="-0.0305"/><!-- toe tab jog, INBOARD (v6) -->
   <!-- MEASURED 2026-07-01 from original NovaSM3 STLs (leg_v5 keeps stock pivots).
        Femur: hfe horn axis (49.5, z10) -> kfe bore (-56.71, z22.02) in

Commit message: leg_v6: stock stance restored (outboard jog) + strap pads
User call, backed by the official assembly: stock stands with straight
vertical legs, feet under the leg columns, semi-wide ~207mm track —
the right geometry for quasi-static v1 bring-up. The inboard-jog
variant (foot 3.3mm from the roll axis, zero holding torque, 84mm
track) is strictly better only with a balance controller; rolling out
to fake a wide stance costs the same torque as stock anyway. Shelved,
documented in the tibia header + memory. d back to 0.0643 everywhere,
tests green.

Also: strap bosses were Ø7 mushrooms overhanging the 3.2mm wall (split
risk under a self-tapper) — replaced with full-width rectangular rim
pads on all three parts.

Co-Authored-By: Claude Fable 5 <noreply@anthropic.com>
Claude-Session: https://claude.ai/code/session_013wnx3m6TJKxLuNtpieRaWF

File: ros2_ws/src/nova_description/urdf/nova.urdf.xacro (robot description, xacro)
@@ -36,12 +36,12 @@
   <xacro:property name="hip_to_upper_x" value="0.0"/>
   <!-- v6 legs (leg_v6/): femur mid-plane 33.8 from haa (coax yoke), femur/
-       tibia coplanar (0), and the toe tab jogs 30.5 INBOARD (v6 rev2 decision
-       2026-07-02 — opposite of stock) so the foot lands 3.3mm from the haa
-       roll axis: near-zero standing roll torque (stock's outboard jog cost
-       ~0.77 N·m/hip holding). Wide stance on demand via hip roll. -->
+       tibia coplanar (0), toe tab jogs 30.5 OUTBOARD (stock stance: straight
+       vertical legs, feet under the leg columns, ~207mm track — right for
+       quasi-static v1). Inboard jog (d=3.3, zero holding torque, 84mm track)
+       evaluated + shelved until a balance controller exists. -->
   <xacro:property name="hip_to_upper_y" value="0.0338"/> <!-- haa axis -> femur mid-plane (v6) -->
   <xacro:property name="hip_to_upper_z" value="-0.0095"/><!-- MEASURED hfe drop below haa -->
   <xacro:property name="upper_to_lower_y" value="0.0"/>  <!-- v6: femur/tibia coplanar -->
-  <xacro:property name="lower_to_foot_y"  value="-0.0305"/><!-- toe tab jog, INBOARD (v6) -->
+  <xacro:property name="lower_to_foot_y"  value="0.0305"/><!-- toe tab jog, outboard (stock stance) -->
   <!-- MEASURED 2026-07-01 from original NovaSM3 STLs (leg_v5 keeps stock pivots).
        Femur: hfe horn axis (49.5, z10) -> kfe bore (-56.71, z22.02) in

Commit message: leg_v6: pose-sweep collision gate + four finds fixed
Adversarial pass hunting known Claude-CAD failure modes. The gate only
checked right-side parts in static pockets — extended to L-mirrors and
actual pose sweeps (knee fold, hip pitch; designed disc interfaces
excluded by axis radius; sampling now seeded/deterministic). Finds:

1. Knee mechanical stop is ~118deg, NOT the hand-computed ~141 (tibia
   pocket-block flank vs fork throat) -> kfe_range 2.2 -> 1.9 rad in
   URDF+IK. Deep-sit stays a v7 offset-plane option.
2. Femur platform corners (r18.6 about the hfe axis) grazed the coax
   bridge -> rounded to r16.1 (servo case corner is r16.05, seat kept).
3. Coax bridge raised 6.9 -> 7.4 (clearance margin).
4. Coax front strap-pad edge sat exactly on the femur rim plane ->
   trimmed to x15.6.
Also: knee-arm diagonal holes are now Ø3.1 close-fit (screws register
the plate; clearance holes let the knee axis wander under cyclic
shear). A text-anchored patch no-op'd AGAIN (hip filter) — caught by
comparing debug vs gate output; block rewritten with an assertion.

build_all now runs the full sweep gate. All clean: 6 pockets 0/21000,
knee to 118deg, hip to +/-86deg. Locomotion tests green.

Co-Authored-By: Claude Fable 5 <noreply@anthropic.com>
Claude-Session: https://claude.ai/code/session_013wnx3m6TJKxLuNtpieRaWF

File: ros2_ws/src/nova_description/urdf/nova.urdf.xacro (robot description, xacro)
@@ -22,5 +22,5 @@
   <xacro:property name="haa_range" value="0.7"/>   <!-- TODO-CAD mechanical travel -->
   <xacro:property name="hfe_range" value="1.5"/>   <!-- TODO-CAD -->
-  <xacro:property name="kfe_range" value="2.2"/>   <!-- TODO-CAD -->
+  <xacro:property name="kfe_range" value="1.9"/>   <!-- sweep-gate: mech stop ~118 deg (tibia flank vs fork throat); 109 sw = margin. Deep-sit = v7 offset-plane option -->
   <!-- ===================== link offsets (m) ===================== -->
   <!-- MEASURED 2026-07-02 from the official Assembly_NOVA_SM3 Fusion share

Commit message: inertials: calibrate density from measured prints (femur 57g)
Printed femur_R shell weighs 57 g (Bambu slicer 56.7 g — estimate trusted).
Real 40%-infill PA6-CF density = 0.712 g/cm3 (was a 0.70-factor / 0.819 g/cm3
guess). Tibia is 25% infill -> 0.586 g/cm3 (51 g slicer). Recomputed every
leg-link inertial (CoM unchanged; mass + inertia scale with density):

  hip   0.087 -> 0.084 kg
  upper 0.131 -> 0.122 kg
  lower 0.131 -> 0.111 kg

Updated compute_inertials.py densities, both URDF (nova.urdf.xacro) and MJCF
(build_mjcf.py LINK_I) sources, regenerated nova.xml. validate_model STANDS,
urdf_sync test green. Legs are ~15-30% lighter than the sim assumed — tightens
sim2real mass fidelity.

Co-Authored-By: Claude Opus 4.8 (1M context) <noreply@anthropic.com>
Claude-Session: https://claude.ai/code/session_01PfnMkwGYyVsyLfTtBhHzYb

File: ros2_ws/src/nova_description/urdf/nova.urdf.xacro (robot description, xacro)
@@ -95,16 +95,14 @@
        URDF's own landmarks — femur STL (106.9,0,0) -> link (0,0,-0.1069)).
        Replaces the old isotropic mass*1e-3 placeholders.
-       ⚠ PROVISIONAL — REFINE BY MEASUREMENT (backlog #5). Mass = solid mesh
-       volume x effective PA6-CF density (1.17 g/cm3 x 0.70 infill) + a 60 g
-       servo box at each pocket. When you WEIGH each printed link, rescale that
-       link's whole <inertial> by measured_mass/computed_mass (CoM unchanged;
-       inertia scales linearly with mass) — one ratio absorbs the density error.
-       ⚠ Servo modeled at the shell centroid; ⚠ LEFT/RIGHT y-sign mirrored via
-       `reflect` (yf=-reflect on com_y/ixy/iyz) — VERIFY THE SIGN IN SIM (matches
-       this file's other gate->URDF sign caveats). base_link stays payload-
-       dominated (~2.8 kg trunk+Jetson+battery+boards+L2/D456); box inertia +
-       measured-CoM refinement still owed.
-       Computed right-leg masses: hip 0.087 upper 0.131 lower 0.131 foot 0.004
-       (vs the old 0.082/0.127/0.130/0.005 estimates — within ~6%). -->
+       CALIBRATED 2026-07-13 from real prints: mesh volume x MEASURED effective
+       density + a 60 g servo box at each pocket. 40%-infill parts (coax/femur/
+       knee_arm/shoulder) = 0.712 g/cm3 (printed femur_R shell 57 g MEASURED,
+       slicer 56.7 g confirmed); the tibia is 25% infill -> 0.586 g/cm3 (51 g
+       slicer). ~15-30% lighter than the old 0.70 guess. Servo box + base_link
+       (~2.8 kg payload, box inertia) unchanged.
+       ⚠ still: Servo modeled at the shell centroid; ⚠ LEFT/RIGHT y-sign mirrored
+       via `reflect` (yf=-reflect on com_y/ixy/iyz) — VERIFY IN SIM.
+       Calibrated right-leg masses: hip 0.084 upper 0.122 lower 0.111 foot 0.004
+       (was 0.087/0.131/0.131 at the 0.70 guess). -->
   <xacro:property name="m_base"  value="2.83"/>
   <!-- base_link: trunk envelope box inertia at m_base (payload-dominated,
@@ -122,7 +120,7 @@
     <inertial>
       <origin xyz="0.00710 ${-reflect*0.02004} 0.00497" rpy="0 0 0"/>
-      <mass value="0.0873"/>
-      <inertia ixx="4.452e-05" iyy="2.275e-05" izz="3.552e-05"
-               ixy="${-reflect*-2.20e-06}" ixz="8.41e-07" iyz="${-reflect*3.81e-06}"/>
+      <mass value="0.0836"/>
+      <inertia ixx="4.099e-05" iyy="2.120e-05" izz="3.255e-05"
+               ixy="${-reflect*-1.91e-06}" ixz="7.32e-07" iyz="${-reflect*3.32e-06}"/>
     </inertial>
   </xacro:macro>
@@ -130,7 +128,7 @@
     <inertial>
       <origin xyz="0.00000 ${-reflect*-0.00653} -0.05067" rpy="0 0 0"/>
-      <mass value="0.1313"/>
-      <inertia ixx="8.366e-05" iyy="7.473e-05" izz="2.907e-05"
-               ixy="${-reflect*-9.47e-10}" ixz="-4.45e-10" iyz="${-reflect*-4.08e-06}"/>
+      <mass value="0.1219"/>
+      <inertia ixx="7.486e-05" iyy="6.649e-05" izz="2.667e-05"
+               ixy="${-reflect*-8.22e-10}" ixz="-3.84e-10" iyz="${-reflect*-3.51e-06}"/>
     </inertial>
   </xacro:macro>
@@ -138,7 +136,7 @@
     <inertial>
       <origin xyz="-0.00054 ${-reflect*-0.01010} -0.06558" rpy="0 0 0"/>
-      <mass value="0.1312"/>
-      <inertia ixx="1.333e-04" iyy="1.225e-04" izz="2.809e-05"
-               ixy="${-reflect*-7.87e-07}" ixz="-1.94e-06" iyz="${-reflect*-1.87e-05}"/>
+      <mass value="0.1110"/>
+      <inertia ixx="1.006e-04" iyy="9.150e-05" izz="2.321e-05"
+               ixy="${-reflect*-5.64e-07}" ixz="-1.39e-06" iyz="${-reflect*-1.34e-05}"/>
     </inertial>
   </xacro:macro>

Commit message: safety: software posture gate is authoritative; firmware loosened to mechanical
The +50 deg hfe fold cap was carried as a per-joint scalar in four places. It is
the riser-skirt bound at ONE posture -- full outboard splay with the knee fully
folded -- and nowhere else: measured, the front leg reaches +70.6 at haa 0, which
is exactly where trot and crawl run. A per-joint scalar CANNOT express a limit
that depends on the other two joints, so holding +50 everywhere clipped every
gait to another posture's worst case.

Split, as designed:
  * CHASSIS constraint  -> posture-aware, upstream:
        nova_locomotion.kinematics.rom_envelope, applied by within_limits()
        and solve_side(), backed off MARGIN_DEG from measured first contact.
  * MECHANICAL travel   -> the per-joint scalars, which is all a scalar can
        honestly represent.

Loosened to mechanical (+86 = leg self-collision 93 deg, LA-19, minus the same
7 deg margin the away-trunk side already used -> a symmetric +-86 window):
    nova.urdf.xacro          hfe_fold  0.873 -> 1.501
    leg_ik.LegParams         hfe_max   0.873 -> 1.501
    nova_ops limits.py       hfe upper   +50 -> +86
    test_joint_map           expectation updated to match

Verified the split actually holds -- hfe +60 at kfe -105 is now INSIDE the
mechanical window, and the gate still refuses it at haa +40 (splayed, would
graze the skirt) while allowing it at haa 0 (clear). That is the behaviour the
scalar could never express.

⚠ ACCEPTED TRADE, stated plainly: the firmware clamp is NO LONGER a backstop
against a riser-skirt strike. It now only stops a command exceeding what the
linkage can do. A skirt strike is prevented solely by the posture gate upstream.
That was the explicit call -- the alternative was clipping every gait to a
posture it never takes.

NOT changed: sim/nova_mjx/build_mjcf.HFE_FOLD stays at 0.873. The MJCF carries no
riser geometry, so there its scalar is the only thing standing in for the
chassis, and widening it would also change the trained walker's environment
(the policy's +-0.4 rad band reaches +57.3, past the current clamp). Wants its
own decision.

155 passed (nova_locomotion + nova_ops + nova_calibration).

Co-Authored-By: Claude Opus 5 (1M context) <noreply@anthropic.com>
Claude-Session: https://claude.ai/code/session_01LbG5HzMixbc1rHytMNrPQt

File: ros2_ws/src/nova_description/urdf/nova.urdf.xacro (robot description, xacro)
@@ -53,5 +53,5 @@
   <xacro:property name="haa_in"   value="0.262"/>  <!-- 15 deg inboard -->
   <xacro:property name="haa_out"  value="0.698"/>  <!-- 40 deg outboard -->
-  <xacro:property name="hfe_fold" value="0.873"/>  <!-- +50 toward trunk (both) -->
+  <xacro:property name="hfe_fold" value="1.501"/>  <!-- +86 toward trunk (both) — MECHANICAL, 2026-07-25. Was +50 (riser-skirt graze); that bound is POSTURE-DEPENDENT (it is the value at full outboard splay + full knee fold only, measured +70.6 at haa 0) and a per-joint scalar cannot express it. Chassis constraint moved to nova_locomotion.kinematics.rom_envelope, enforced per posture by within_limits/solve_side. 86 = leg self-collision 93 (LA-19) minus the same 7deg margin hfe_ext uses -> symmetric window. -->
   <xacro:property name="hfe_ext"       value="1.501"/>  <!-- -86 away, REAR legs -->
   <xacro:property name="hfe_ext_front" value="1.501"/>  <!-- -86 away, FRONT legs — #47: head clearance is NOT the binding constraint (measured), leg self-collision (LA-19, 93deg) is; matches hfe_ext -->
