Commit message: safety: move the posture gate to the choke point, then re-loosen firmware
Acting on the review of the previous commit, which found that loosening
limits.py to mechanical had opened a hole I created.

THE REGRESSION: the posture gate lived only in nova_locomotion.solve_side --
the GAIT path. nova_calibration's servo_homing and actuator_char publish
/joint_commands DIRECTLY and never touch it. limits.py was their only chassis
protection, and I had just widened it +50 -> +86. Homing is the first thing that
runs on real hardware, and its whole job is driving joints toward hard stops.

Sequence, in order:
  1. limits.py reverted to +50 immediately.
  2. Review gaps closed by re-measuring, not by argument:
     S2  positive kfe was never swept -- every kfe > 0 extrapolated from the
         kfe=0 row. Now swept to +109. (The extrapolation happened to be
         right: the bound saturates at 76.9 for kfe >= -25. Measured now.)
     S3  only FL and RL were swept, right side ASSUMED mirror-identical.
         All four now swept and stored per-leg. Measured max L/R asymmetry
         across every cell: 0.0 deg -- the assumption held, but it is
         verified rather than assumed, and the table is per-leg either way.
  3. rom_envelope moved nova_locomotion/kinematics -> nova_ops/safety_envelope.
     It had to: nova_locomotion.node already imports nova_ops, so nova_ops ->
     nova_locomotion would have been a genuine cycle. It also belongs next to
     limits.py -- same kind of artifact.
  4. wrapper.publish() now applies hfe_bounds() per leg BEFORE the per-joint
     scalars. HAA SIGN IS UNKNOWN in the servo command frame until homing fills
     HAA_INBOARD_SIGN, so both interpretations of a commanded haa are evaluated
     and the tighter taken -- the same conservative posture limits.py already
     takes for haa itself.
  5. Only then limits.py re-loosened to mechanical +86.

Locked by two new tests: a splayed+folded command IS clamped while the same
fold at neutral haa passes untouched (the behaviour no scalar can express), and
the bound is identical for either sign of a commanded haa.

157 passed.

Co-Authored-By: Claude Opus 5 (1M context) <noreply@anthropic.com>
Claude-Session: https://claude.ai/code/session_01LbG5HzMixbc1rHytMNrPQt

File: ros2_ws/src/nova_description/urdf/nova.urdf.xacro (robot description, xacro)
@@ -53,5 +53,5 @@
   <xacro:property name="haa_in"   value="0.262"/>  <!-- 15 deg inboard -->
   <xacro:property name="haa_out"  value="0.698"/>  <!-- 40 deg outboard -->
-  <xacro:property name="hfe_fold" value="1.501"/>  <!-- +86 toward trunk (both) — MECHANICAL, 2026-07-25. Was +50 (riser-skirt graze); that bound is POSTURE-DEPENDENT (it is the value at full outboard splay + full knee fold only, measured +70.6 at haa 0) and a per-joint scalar cannot express it. Chassis constraint moved to nova_locomotion.kinematics.rom_envelope, enforced per posture by within_limits/solve_side. 86 = leg self-collision 93 (LA-19) minus the same 7deg margin hfe_ext uses -> symmetric window. -->
+  <xacro:property name="hfe_fold" value="1.501"/>  <!-- +86 toward trunk (both) — MECHANICAL, 2026-07-25. Was +50 (riser-skirt graze); that bound is POSTURE-DEPENDENT (it is the value at full outboard splay + full knee fold only, measured +70.6 at haa 0) and a per-joint scalar cannot express it. Chassis constraint moved to nova_ops.safety_envelope.rom_envelope, enforced per posture at the choke point by safety_envelope.wrapper (every publisher) and by within_limits/solve_side (gait path). 86 = leg self-collision 93 (LA-19) minus the same 7deg margin hfe_ext uses -> symmetric window. -->
   <xacro:property name="hfe_ext"       value="1.501"/>  <!-- -86 away, REAR legs -->
   <xacro:property name="hfe_ext_front" value="1.501"/>  <!-- -86 away, FRONT legs — #47: head clearance is NOT the binding constraint (measured), leg self-collision (LA-19, 93deg) is; matches hfe_ext -->
