Commit message: Disprove the stair 'hardware wall'; fix 3 latent kinematics bugs; posture-aware chassis ROM gate (#147)
* docs: v9 imitation-crawl spec — scripted expert -> BC -> RL fine-tune (expert-first premise gate)

* sim: scripted crawl-climb controller (v9 imitation expert — premise gate)

Whole-body crawl-climb: validated leg IK + crawl schedule (CRAWL_OFFSETS/DUTY)
+ foothold planner reading treads off the collision surface + CoM-shift sway
+ body pitch, via body-pose control with a forward body lean for propulsion.

Premise gate FAILS: stable forward crawl reaches the first riser (front foot
onto tread 1, 2cm) but does NOT ascend >=2 risers. Level 0.25 stalls at the
riser (stable, up_z 0.976); level 0.5 topples at the 4cm step. No stable
operating point climbs 2 risers (gentle stalls, aggressive topples) — the
position-servo torque cannot lift the loaded body up a step. Report +
video/frames/traces in .superpowers/sdd (gitignored) and climber_out/.

Co-Authored-By: Claude Opus 4.8 <noreply@anthropic.com>
Claude-Session: https://claude.ai/code/session_01Kkc2GgdBWpBZs6xtVHMZ1Y

* sim: disprove the stair "hardware wall" + fix three IK defects (#142)

The servo-upgrade question ("buy 8x 30 kgf.cm femur/tibia?") is answered
NO, measured. Scaling hfe/kfe stall torque 1.63/2.72/4.0x, with kp matched
so it is not a detuning artifact, never climbed and made things worse:
travel collapsed 37 -> 5 cm and falls came earlier. Static capacity says
why -- 42.0 N per stance leg vs a 13.4 N share (3.13x), 552 N at the best
pose, and 8.5x lift-power margin. Torque was never the binding constraint.

New probes:
  probe_lift_force.py     force capacity + the hfe fold-cap step-up budget
  probe_lift_envelope.py  true envelope: any force direction (the old
                          pure-vertical assumption understated by 70%),
                          full-workspace sweep, torque-speed-derated power
  probe_posture_search.py joint search over body height / pitch / abduction
                          -- 13.59 cm of swing clearance available vs the
                          5.69 cm the climber's fixed-height plan uses
  render_knee_configs.py  side-by-side knee-configuration views

ik_action had three defects, all fixed:
  1. leg_ik.solve_side is documented as THE ONE MIRRORING BOUNDARY, and
     ik_action bypassed it -- right-leg haa was never negated, so FR/RR
     drove the WRONG WAY on every CoM sway and abduction. Dormant at the
     haa=0 default pose, active exactly when the hips do something. Fixing
     it turned a flat-ground fall at step 598 into a full stable episode
     and cut stairs n_unreach 4362 -> 268.
  2. joint limits were not checked at all -- IK "succeeded" out of range,
     MuJoCo clamped at the stop, the foot silently missed its target.
  3. the knee branch was hard-coded knee_forward=False, locking out the
     branch the best-clearance posture wants. Both are tried now, with
     hysteresis (a mid-motion flip swings the leg through full extension).

Climber also gains --eff-scale/--kp-scale/--swing-abduct/--abduct-climb/
--splay/--knee-config, a torque-saturation readout, and an approach-pad
guard (round 1 was confounded: 900 steps only crossed the 50 cm flat pad
and never reached a riser, so the FAIL measured walking speed).

Measured, not assumed: swing-phase abduction helps (fall@725 -> survived
3500, 5x travel); global stance splay HURTS (n_unreach 4362 -> 6387).
n_outband reports that 47-65% of the expert's joint commands fall outside
the +-0.4 rad band a tanh policy can express -- a problem for the v9
imitation premise independent of whether the expert climbs.

Co-Authored-By: Claude Opus 5 (1M context) <noreply@anthropic.com>
Claude-Session: https://claude.ai/code/session_01LbG5HzMixbc1rHytMNrPQt

* locomotion: correct knee config to TRANSLATED, raise choreo keyframes

KNEE_FORWARD read {FL: True, FR: True, RL: False, RR: False}, recording an
"X-CONFIG decided 2026-07-06" that was NEVER BUILT. The robot is the
TRANSLATED layout -- all four knees bend backward -- and the MJX sim always
matched it (DEFAULT_POSE kfe -1.2 on every leg). The stale value commanded
the FRONT knees FORWARD, so controller.gait_pose would have driven the front
legs to a mirrored stance on first stand. Now all four False.

Verified by sim/nova_mjx/render_knee_configs.py, which measures each knee
against the hip->foot chord: -66.0 mm (backward) on all four legs.

Knee config is pure software -- CAD femur/tibia are mirrored left/right
only, never front/rear -- so nothing physical had to change.

CONSEQUENCE, and it is not free. Translated crouches by folding the FRONT
legs TOWARD the trunk, into the riser skirt (hfe_max +50 deg; chassis gate
2026-07-06 measured tibia-flank contact from ~+55). The old lie/crouch
depths need +61.3 and +57.4 deg, both past the cap -- solve_side's
FRONT_LEGS clamp fired and the foot landed 27 mm off target. Under X-config
the front legs took the elbow-forward branch and folded AWAY from the trunk
into the -86 deg window, which is where that layout's crouch margin came
from; translated forfeits it.

Keyframes raised inside the cap with margin:
  crouch 0.150 -> 0.1755  (front hfe +47.0 deg, 3.0 deg of margin)
  lie    0.140 -> 0.1708  (front hfe +49.0 deg, 1.0 deg of margin)
  stand  0.180 unchanged  (+45.1 deg)
All three are now IK-consistent: the clamp never fires, foot error 0.0000 mm.

Crouch travel is 4.00 -> 0.92 cm. lie/crouch/stand now sit within 9 mm of
each other, so the sit/stand choreography is functionally flat. Recovering
it needs either a front/rear ASYMMETRIC crouch (pure software -- only the
front pair is skirt-limited; the rear folds away from the trunk and keeps
its full -86 room, which is also how a dog sits) or a riser-skirt trim, the
same part that caps stair step-up. Both left open.

test_x_config_rear_knees_mirrored -> test_translated_config_all_knees_backward.
83 passed in nova_locomotion; 72 in nova_ops + nova_calibration.

Co-Authored-By: Claude Opus 5 (1M context) <noreply@anthropic.com>
Claude-Session: https://claude.ai/code/session_01LbG5HzMixbc1rHytMNrPQt

* sim: sit / belly-down poses, stand-up recovery, and sit descent timing (#142)

choreo/stand.py can only express symmetric feet-under-hips poses, which routes
100% of a crouch into hfe fold -- the one direction the riser skirt caps at +50.
That is what collapsed the translated-knee crouch envelope to 0.92 cm. The robot
has two ways down that never approach the cap, and both are measured here:

  render_sit_poses.py  commands backlog #15's sit (haa +40/hfe +40/kfe -90) and
                       lets it settle under gravity through the real servos.
                       ASYMMETRIC SIT: trunk 9.85 cm, nose-up 24.3 deg, rear
                       belly down, 10 deg of skirt margin (choreo 'lie' gets
                       17.08 cm and 1 deg). BELLY DOWN: trunk 6.42 cm, level.
                       Foot protraction is the other route -- hip reaches
                       2.00 cm at foot x +14 cm with hfe -21 deg, running AWAY
                       from the cap into the unused -86 side.

  probe_standup.py     can it LEAVE those poses? 6/6 yes -- both poses, blends
                       1.5/3/6 s, reach full 17.6 cm without rolling, on a plain
                       joint-space min-jerk blend with no balance controller.
                       3 s is the sweet spot (16.7% torque saturation vs 33.3%
                       at 1.5 s for no height gain). CAVEAT: recovery drags the
                       feet ~9 cm inboard against mu=1.2 -- fine in sim, may bind
                       on carpet. A staggered lift-and-place is the robust form.

  probe_sitdown.py     how long may the fault path keep servos powered? The
                       firmware slew limiter (20 raw/broadcast @ 100 Hz =
                       175.8 deg/s) floors the sit at 227 ms, but free fall over
                       the same 11.2 cm drop is 151 ms -- so at the limiter the
                       "controlled" sit is nearly a drop and lands at 3.16x
                       static weight with servos railed 67% of the time.
                       MEASURED ANSWER: ~1 s (1.65x static, 8.3% saturation).
                       An earlier 3 s estimate was borrowed from the stand-up
                       and was 3x too conservative.

Co-Authored-By: Claude Opus 5 (1M context) <noreply@anthropic.com>
Claude-Session: https://claude.ai/code/session_01LbG5HzMixbc1rHytMNrPQt

* choreo: per-leg keyframes + sit/down poses (gated on homing calibration)

KEYFRAMES returned ONE shared (x, y, z) for all four legs with x = 0 and
haa = 0 -- "feet under hips". That rule is what collapsed the translated-knee
crouch envelope to 0.92 cm: with the foot pinned under the hip, ALL of a height
change must come out of hfe fold, and fold is the one direction the riser skirt
caps at +50 deg. Freeing the foot removes the cap as the binding constraint --
min hip height goes 16.85 -> 2.00 cm, because a foot placed FORWARD drives hfe
NEGATIVE (phi = atan2(-x, -z)) into the unused -86 deg side.

KEYFRAMES is now per-leg, so a pose may be front/rear asymmetric. Added two
JOINT-space poses from backlog #15's controlled-limp angles (haa +40 / hfe +40 /
kfe -90) -- they are defined by where the CHASSIS lands, not by a foot target:
  down  all four splayed+folded, belly onto the skid rails
  sit   dog sit: REAR splayed+folded, FRONT holding stand -> nose-up ~24 deg

Both verified in sim before being written here: settled under gravity through
the real position servos (render_sit_poses.py -- sit trunk 9.85 cm with 10 deg
of skirt margin vs 'lie' at 17.08 cm and 1 deg), and RECOVERABLE -- stand-up
succeeds 6/6 from both, no balance controller needed (probe_standup.py).

sit/down deliberately RAISE for now. They need ~40 deg OUTBOARD haa, and
LegParams.haa_range is an intentional conservative symmetric +-15 deg (the
chassis gate's INBOARD cap) that stays symmetric until
nova_ops.safety_envelope.limits.HAA_INBOARD_SIGN is filled -- that sign is the
inboard direction in the SERVO COMMAND frame and is unknowable until homing
watches a real servo move. limits.py already says splay choreography is the
reason to fill it. The error names the exact unlock rather than failing
generically, so nothing emits a pose the runtime would silently clamp -- the
failure mode that just put lie/crouch 27 mm off target.

83 passed.

Co-Authored-By: Claude Opus 5 (1M context) <noreply@anthropic.com>
Claude-Session: https://claude.ai/code/session_01LbG5HzMixbc1rHytMNrPQt

* chassis+ik: rear hip placement was a REFLECTION; per-END hfe windows measured

check_fit's crouch sweep placed the REAR hip with the fore-aft sign inside the
ROTATION as well as the translation ([0, end, 0, end*HIP_FA]), making the rear
placement a reflection: det(S2T @ MIR) = -1 rear vs +1 front. A reflection is
not a placement any physical part can take. leg_v6/ ships only LEFT/RIGHT
variants (coax/coax_L, femur/femur_L, tibia/tibia_L, shoulder_plate/_L) -- there
is no front/rear part, so the rear leg is the SAME part in the SAME orientation
translated to -HIP_FA, which is what sim/nova_mjx/build_mjcf.py models.

Consequence of the old mirror: front and rear swept IDENTICAL volumes (FR and RR
returned byte-identical hit counts for every pose), so the gate could never
produce a per-END answer. Its "+50 toward-trunk fold, BOTH ends" was ONE
measurement reported as two.

With the rear placement corrected the gate FAILS, and the map is an exact mirror
(union over haa x kfe x target):
    hfe   FRONT                      REAR
    -86   clean                      pack,pocket,rails,RISER
    -45   clean                      pack,pocket,rails
    +45   pack,pocket,rails          clean
    +55   pack,pocket,rails,RISER    clean
    +86   pack,pocket,rails,RISER    clean
=> FRONT [hfe_min, +50], REAR [-50, -hfe_min]. Skirt contact +55 front, -55 rear.

So the asymmetric hfe window keys on LEG POSITION, not the knee branch: which
SIGN of canonical hfe points toward the trunk depends on where the leg is
mounted. within_limits keyed it on knee_forward, which silently gave EVERY leg
the REAR window once KNEE_FORWARD became all-False -- certifying front poses out
to +86 against a skirt that contacts at +55. Fixed. Unknown leg now gets the
conservative INTERSECTION instead of a permissive default.

solve_side: REAR legs had NO runtime clamp at all (issue #47 was front-only, on
the belief the skirt cap was front-only too). Added, to the mirror window.

⚠ FOUR TESTS LEFT FAILING ON PURPOSE -- they report a real, unfixed blocker:
under the built TRANSLATED config both primary gaits drive the FRONT legs into
the riser skirt.
    trot   FL/FR hfe +34.5..+59.4  (cap +50, contact +55)  -> 4.4 deg past contact
    crawl  FL/FR hfe +36.4..+57.0                          -> 2.0 deg past contact
    body_pose likewise
The excursion magnitude is unchanged and was always ~59 deg; the knee-config
correction flips its SIGN, and on a front leg that sign points into the skirt.
The old test_trot hid this by solving knee_forward=True (the elbow-FORWARD
branch the robot does not use), which put the same excursion at -59.4 deg,
comfortably inside. Now solved with KNEE_FORWARD[leg]. Fixing it is a gait
retune (or a skirt trim) -- a design decision, not a test edit.

Co-Authored-By: Claude Opus 5 (1M context) <noreply@anthropic.com>
Claude-Session: https://claude.ai/code/session_01LbG5HzMixbc1rHytMNrPQt

* ik: posture-aware chassis hfe bound, measured (replaces the worst-case scalar)

The chassis ROM was one scalar -- "hfe toward-trunk fold +50 deg" -- but the
constraint is 3-dimensional: how far the leg folds before the tibia flank reaches
the riser skirt depends on how far the hip is splayed and the knee folded AT THE
SAME TIME. Applying one worst-case number at every posture failed poses that are
geometrically clear, and would have cost real stride to "fix".

hardware/cad/chassis/hfe_envelope.py sweeps the contact-free hfe interval per leg
END over a (haa x kfe) grid, against every target the crouch sweep uses (riser,
battery pocket, pack, skid rails, head), with check_fit's rear hip placement
corrected. Emits rom_envelope_table.py; a copy lives in the kinematics package.

    FRONT  haa +40 (full outboard splay), kfe -109  ->  +51.7   <- the old scalar
    FRONT  haa   0                      , kfe -109  ->  +70.6   <- where gaits run
    FRONT  haa   0                      , kfe  -25  ->  +76.9
    REAR   haa   0                                  ->  -80.1

So +50 was very nearly the true worst case over legal haa (+51.7) -- correct, but
applied everywhere. At haa 0 the real front bound is +70.6, so the trot's +59.4
excursion has ~11 deg of margin and never needed retuning. The earlier "gaits
drive the front legs into the skirt" reading was comparing against a posture the
gaits never take.

within_limits and solve_side now take the bound from rom_envelope.hfe_bounds(),
intersected with the leg's own mechanical travel. Lookup is CONSERVATIVE: a query
between cells takes the tightest bound of the enclosing cells, outside the grid
clamps to the edge, exact grid hits do not widen, and an unknown leg gets the
FRONT-REAR intersection.

The haa grid is fine (-15/-12/-10/-8/-5) across the inboard belly-pack edge: the
bound collapses hard once the leg rolls under the pack, and a coarse 10-deg grid
dragged that collapsed neighbour into every conservative bracket just inside the
legal cap -- which is what made body_pose fail at haa -10.01.

Also corrects my own earlier guess: I had inferred the REAR window was the exact
mirror [-50, +86]. Measured, it is ~[-79, +95]. The coarse sweep only bracketed
it between -86 and -45.

⚠ DOWNSTREAM SCALARS NOT RAISED -- deliberately. LegParams.hfe_max, the xacro
hfe_fold, build_mjcf.HFE_FOLD and nova_ops limits.py still carry +50, so the
RUNTIME still clamps there. Regenerating them from this table is a
hardware-affecting change and wants its own review.

83 passed in nova_locomotion; 72 in nova_ops + nova_calibration.

Co-Authored-By: Claude Opus 5 (1M context) <noreply@anthropic.com>
Claude-Session: https://claude.ai/code/session_01LbG5HzMixbc1rHytMNrPQt

* ik: back the posture gate off first contact by a clearance margin

The envelope table is raw geometry -- the angle at which the leg TOUCHES the
chassis. A gate that permits poses right up to that boundary permits grazing.
The gate exists to refuse a posture for coming NEAR the body, so hfe_bounds()
now backs off MARGIN_DEG from every measured edge.

5 deg is not a new invention: it is the convention the project already used --
the chassis gate measured front skirt contact at ~+55 and published the cap
as +50. Applying it in the lookup rather than baking it into the table keeps
the measurement a measurement and the margin tunable in one place.

Effect at the postures that matter:
    FRONT haa   0, kfe -105  ->  +64.7   (raw +70.6 (was) - 5, then bracketing)
    FRONT haa +40, kfe -105  ->  +46.7
    REAR  haa   0            ->  -75.1
Trot's front worst case is +59.4 and crawl's +57.0, so both still clear the
gate -- with 5.3 and 7.7 deg of margin respectively, rather than sitting on a
contact boundary.

A cell whose margin exceeds its own width collapses to a point rather than
inverting, so an over-tight posture is refused outright instead of silently
producing lo > hi.

155 passed (nova_locomotion + nova_ops + nova_calibration).

Co-Authored-By: Claude Opus 5 (1M context) <noreply@anthropic.com>
Claude-Session: https://claude.ai/code/session_01LbG5HzMixbc1rHytMNrPQt

* safety: software posture gate is authoritative; firmware loosened to mechanical

The +50 deg hfe fold cap was carried as a per-joint scalar in four places. It is
the riser-skirt bound at ONE posture -- full outboard splay with the knee fully
folded -- and nowhere else: measured, the front leg reaches +70.6 at haa 0, which
is exactly where trot and crawl run. A per-joint scalar CANNOT express a limit
that depends on the other two joints, so holding +50 everywhere clipped every
gait to another posture's worst case.

Split, as designed:
  * CHASSIS constraint  -> posture-aware, upstream:
        nova_locomotion.kinematics.rom_envelope, applied by within_limits()
        and solve_side(), backed off MARGIN_DEG from measured first contact.
  * MECHANICAL travel   -> the per-joint scalars, which is all a scalar can
        honestly represent.

Loosened to mechanical (+86 = leg self-collision 93 deg, LA-19, minus the same
7 deg margin the away-trunk side already used -> a symmetric +-86 window):
    nova.urdf.xacro          hfe_fold  0.873 -> 1.501
    leg_ik.LegParams         hfe_max   0.873 -> 1.501
    nova_ops limits.py       hfe upper   +50 -> +86
    test_joint_map           expectation updated to match

Verified the split actually holds -- hfe +60 at kfe -105 is now INSIDE the
mechanical window, and the gate still refuses it at haa +40 (splayed, would
graze the skirt) while allowing it at haa 0 (clear). That is the behaviour the
scalar could never express.

⚠ ACCEPTED TRADE, stated plainly: the firmware clamp is NO LONGER a backstop
against a riser-skirt strike. It now only stops a command exceeding what the
linkage can do. A skirt strike is prevented solely by the posture gate upstream.
That was the explicit call -- the alternative was clipping every gait to a
posture it never takes.

NOT changed: sim/nova_mjx/build_mjcf.HFE_FOLD stays at 0.873. The MJCF carries no
riser geometry, so there its scalar is the only thing standing in for the
chassis, and widening it would also change the trained walker's environment
(the policy's +-0.4 rad band reaches +57.3, past the current clamp). Wants its
own decision.

155 passed (nova_locomotion + nova_ops + nova_calibration).

Co-Authored-By: Claude Opus 5 (1M context) <noreply@anthropic.com>
Claude-Session: https://claude.ai/code/session_01LbG5HzMixbc1rHytMNrPQt

* safety: move the posture gate to the chok

File: ros2_ws/src/nova_description/urdf/nova.urdf.xacro (robot description, xacro)
@@ -53,5 +53,5 @@
   <xacro:property name="haa_in"   value="0.262"/>  <!-- 15 deg inboard -->
   <xacro:property name="haa_out"  value="0.698"/>  <!-- 40 deg outboard -->
-  <xacro:property name="hfe_fold" value="0.873"/>  <!-- +50 toward trunk (both) -->
+  <xacro:property name="hfe_fold" value="1.501"/>  <!-- +86 toward trunk (both) — MECHANICAL, 2026-07-25. Was +50 (riser-skirt graze); that bound is POSTURE-DEPENDENT (it is the value at full outboard splay + full knee fold only, measured +70.6 at haa 0) and a per-joint scalar cannot express it. Chassis constraint moved to nova_ops.safety_envelope.rom_envelope, enforced per posture at the choke point by safety_envelope.wrapper (every publisher) and by within_limits/solve_side (gait path). 86 = leg self-collision 93 (LA-19) minus the same 7deg margin hfe_ext uses -> symmetric window. -->
   <xacro:property name="hfe_ext"       value="1.501"/>  <!-- -86 away, REAR legs -->
   <xacro:property name="hfe_ext_front" value="1.501"/>  <!-- -86 away, FRONT legs — #47: head clearance is NOT the binding constraint (measured), leg self-collision (LA-19, 93deg) is; matches hfe_ext -->
