Commit message: cad review: rear hip is a 180° yaw, not a translation — and the posture table knows it
The chassis gate placed the rear leg as a pure translation of the front (the
2026-07-25 "unmirrored rear" fix). It cannot be: shoulder.scad is ONE part at
both trunk ends and its flange bolts to the trunk END FACE (±63.5 from
trunk.stl, +77.7 flange = the ±141.2 hip station), so the rear crossmember is
the front placement YAWED 180° about Z. Under a translation the rear flange
lands at x −218.9 — 155 mm behind the trunk it bolts to — and the rear coax's
horn face at −123.4 against a rear shoulder whose horn plane the SAME gate puts
at −158.9. The gate was bolting a translated leg onto a yawed shoulder.

Fixed in chassis/check_fit.py coax_to_trunk_bases() (front bases byte-identical;
only the two rear bases move) and preview_assembly.py, with the derivation in
place. Verified against the meshes: all four corners now land their coax horn
face on their own shoulder's horn plane, and the hfe axis sits 11.6 mm toward
the trunk at both ends (±129.6, not −152.8 at the rear).

Consequences recorded, not silently patched:

* rom_envelope_table.py's REAR rows are invalid — and since limits.py loosened
  the hfe scalar to mechanical ±86 in the same batch, that table is the sole
  chassis protection. Re-measured with the fix (same targets + 5 mm proximity,
  box-model servo stand-in, 2° scan; FRONT rows reproduce the shipped table to
  ~2°, which validates the method): every rear cell equals its front
  counterpart — [−94,+66] at haa 0/kfe −109, [−94,+14] at haa −15/kfe −109 —
  where the shipped rear rows carry a flat [−77.2,+95] at all ten kfe values.
  Regeneration needs the real servo.stl, so it is left to the owner, along with
  pinning the leg-local→canonical hfe SIGN for the yawed rear hips (their local
  +hfe is the opposite world rotation from the front's; same class as #153/#155).
* leg chirality pairs DIAGONALLY (front +y = R, rear +y = L). leg_v6/README.md's
  "front and rear are the same parts translated" corrected, with the corner
  table and the FL↔RR / FR↔RL labelling note.
* URDF body_half_x / MJX MOUNT.x 0.1412 is the STOCK hfe station (dimensions.md's
  hip grid mixes the haa horn for lateral with the hfe axis for fore-aft — legal
  for stock, not for v6). Built pitch axes are at ±129.6, so the modeled stance
  is 23.2 mm longer fore-aft than the robot. Flagged in dimensions.md, the
  xacro, build_mjcf.py and the backlog; NOT changed — it moves the geometry every
  trained policy was fit to.

Also: full review in docs/cad-review-2026-07-26.md (incl. what verified healthy —
the servo-independent leg gates and mesh_health are green on the committed STLs),
the wheel-BCD head protrusion (~0.9 mm proud) and the fastener-schedule's stale
"5th center hole" claim (removed under #51), the anti-rot-rib vs drop-in
acceptance tension, and a stale-comment batch (femur SUB_X1, Ø24→Ø21.5 window,
Ø7→Ø9.5 idler relief, coax's pre-rev-3 cap-ridge note). No geometry changed, so
the committed STLs stay valid.

Co-Authored-By: Claude Opus 5 <noreply@anthropic.com>
Claude-Session: https://claude.ai/code/session_01731pwtuXBTtZei6dq31Qmv

File: ros2_ws/src/nova_description/urdf/nova.urdf.xacro (robot description, xacro)
@@ -65,5 +65,18 @@
        the tibia S-curve puts the foot 30.5 mm outboard of kfe.
        Total haa->foot lateral = 64.3 mm = LegParams.hip_offset. -->
-  <xacro:property name="body_half_x" value="0.1412"/> <!-- MEASURED half hip-grid length -->
+  <!-- ⚠ OPEN (CAD review 2026-07-26): body_half_x + hip_to_upper_x below are a
+       STOCK-assembly pair. 141.2 is the stock HFE-axis fore-aft station, which
+       is why hip_to_upper_x = 0 is exact for stock (the haa axis is fore-aft
+       parallel, so its own station along that axis is a kinematic no-op).
+       leg_v6 moved it: shoulder.scad puts the haa station at ±141.2 (trunk end
+       face ±63.5 + 77.7 flange) and coax.scad puts the hfe axis 11.6 mm TOWARD
+       THE TRUNK of it, at both ends -> real pitch-axis spacing 259.2, not
+       282.4. So this model's stance is 23.2 mm longer fore-aft than the built
+       robot (same error in sim/nova_mjx/build_mjcf.py MOUNT/HAA_TO_HFE).
+       Fix is either body_half_x 0.1296 or hip_to_upper_x ∓0.0116 — NOT changed
+       here: it shifts every trained policy's geometry and is a B2/gait-lane
+       call. Details: hardware/cad/dimensions.md "Hip grid" +
+       docs/cad-review-2026-07-26.md §2. -->
+  <xacro:property name="body_half_x" value="0.1412"/> <!-- MEASURED half hip-grid length (⚠ stock hfe station, see above) -->
   <xacro:property name="body_half_y" value="0.0390"/> <!-- MEASURED half hip-grid width  -->
   <xacro:property name="mount_z"     value="0.0380"/> <!-- hip row above chassis-mesh origin; ⚠ REVIEW-visual (trunk-node bbox polluted by children) -->
