Commit message: B2: hip offsets + body mount grid measured from official A360 assembly
Source: the Assembly_NOVA_SM3 Fusion share embedded on novaspotmicro.com
— queried the viewer instance tree for world transforms; the 25t
servo-horn instances mark every joint axis exactly.

- hip grid 282.4 x 78.1 mm (body_half_x/y 0.1412/0.0390), hips ~38mm
  above chassis-mesh origin (mount_z, flagged REVIEW-visual)
- lateral chain haa->foot = 24.6 + 9.2 + 30.5 = 64.3 mm: URDF now
  carries per-joint y offsets (new upper_to_lower_y / lower_to_foot_y,
  reflect-aware in leg macro); IK hip_offset = 0.0643 folds the sum
- test_urdf_sync now asserts d == sum of URDF lateral offsets
- assembly cross-checks femur at 105.9 vs 106.9 bore-metric (kept)

Remaining TODO-CAD: joint ranges, masses/inertias.

Co-Authored-By: Claude Fable 5 <noreply@anthropic.com>
Claude-Session: https://claude.ai/code/session_013wnx3m6TJKxLuNtpieRaWF

File: ros2_ws/src/nova_description/urdf/leg.macro.xacro (robot description, xacro)
@@ -54,5 +54,5 @@
       <parent link="${leg}_upper"/>
       <child  link="${leg}_lower"/>
-      <origin xyz="${upper_to_lower_x} 0 ${upper_to_lower_z}" rpy="0 0 0"/>
+      <origin xyz="${upper_to_lower_x} ${reflect*upper_to_lower_y} ${upper_to_lower_z}" rpy="0 0 0"/>
       <axis xyz="0 1 0"/>
       <limit lower="${-kfe_range}" upper="${kfe_range}"
@@ -72,5 +72,5 @@
       <parent link="${leg}_lower"/>
       <child  link="${leg}_foot"/>
-      <origin xyz="${lower_to_foot_x} 0 ${lower_to_foot_z}" rpy="0 0 0"/>
+      <origin xyz="${lower_to_foot_x} ${reflect*lower_to_foot_y} ${lower_to_foot_z}" rpy="0 0 0"/>
     </joint>
     <link name="${leg}_foot">

File: ros2_ws/src/nova_description/urdf/nova.urdf.xacro (robot description, xacro)
@@ -24,11 +24,19 @@
   <xacro:property name="kfe_range" value="2.2"/>   <!-- TODO-CAD -->
   <!-- ===================== link offsets (m) ===================== -->
-  <!-- TODO-CAD: every value below is a placeholder SpotMicro-class guess. -->
-  <xacro:property name="body_half_x" value="0.10"/>  <!-- TODO-CAD half trunk length -->
-  <xacro:property name="body_half_y" value="0.05"/>  <!-- TODO-CAD half trunk width  -->
-  <xacro:property name="mount_z"     value="0.0"/>   <!-- TODO-CAD hip row height -->
-  <xacro:property name="hip_to_upper_x" value="0.0"/>    <!-- TODO-CAD -->
-  <xacro:property name="hip_to_upper_y" value="0.045"/>  <!-- TODO-CAD coax horn -> femur axis -->
-  <xacro:property name="hip_to_upper_z" value="0.0"/>    <!-- TODO-CAD -->
+  <!-- MEASURED 2026-07-02 from the official Assembly_NOVA_SM3 Fusion share
+       (A360 viewer instance-tree world transforms; servo-horn instances mark
+       the joint axes). Numbers + method: hardware/cad/dimensions.md §6.
+       Hip grid: haa axes 282.4 mm fore-aft x 78.1 mm lateral; hfe sits
+       24.6 mm outboard + 9.5 mm below haa; kfe a further 9.2 mm outboard;
+       the tibia S-curve puts the foot 30.5 mm outboard of kfe.
+       Total haa->foot lateral = 64.3 mm = LegParams.hip_offset. -->
+  <xacro:property name="body_half_x" value="0.1412"/> <!-- MEASURED half hip-grid length -->
+  <xacro:property name="body_half_y" value="0.0390"/> <!-- MEASURED half hip-grid width  -->
+  <xacro:property name="mount_z"     value="0.0380"/> <!-- hip row above chassis-mesh origin; ⚠ REVIEW-visual (trunk-node bbox polluted by children) -->
+  <xacro:property name="hip_to_upper_x" value="0.0"/>
+  <xacro:property name="hip_to_upper_y" value="0.0246"/> <!-- MEASURED haa axis -> femur horn plane -->
+  <xacro:property name="hip_to_upper_z" value="-0.0095"/><!-- MEASURED hfe drop below haa -->
+  <xacro:property name="upper_to_lower_y" value="0.0092"/><!-- MEASURED hfe->kfe outboard shift -->
+  <xacro:property name="lower_to_foot_y"  value="0.0305"/><!-- MEASURED tibia S-curve outboard shift -->
   <!-- MEASURED 2026-07-01 from original NovaSM3 STLs (leg_v5 keeps stock pivots).
        Femur: hfe horn axis (49.5, z10) -> kfe bore (-56.71, z22.02) in

Commit message: improvement batch 1: backlog notes + insert bosses + breakaway fuses + BOM + gate-ROM URDF
docs/improvement-backlog.md: all 13 review items with status/triggers.

Implemented now:
#1 shoulder lower trunk-bolt insert bosses (upper bores were already
   backed by the shear webs; lower pair padded 4->7) — prying SF 2.5->~5.
   Chassis + leg gates green.
#2 breakaway fuses = NYLON M3x10 screws at the L2-mast deck flange and
   D456 bracket row (zero CAD): mounts pop at ~10 N.m faceplant instead
   of the sensor/riser dying, both stay cable-tethered. Hand-tight only.
#3 BOM: nylon M3 pack, M3 washers for every stock-shell bearing head,
   M3x14 csk + nylocs for the rev4 flange feet.
#13 URDF: gate-derived ROM replaces placeholders — haa asymmetric per
   side (inboard 15 / outboard 40, reflect-conditional), hfe -86..+50
   (sign mapping flagged VERIFY IN SIM), kfe +/-109 (already done);
   masses = CAD-volume estimates (total 4.206 kg, weigh at next print
   batch). xacro processes clean; asymmetry verified in output. limits.py
   gets a loud note: firmware haa +/-45 default is LOOSER than the gate's
   15-deg inboard cap — tighten in the firmware lane (#9) via the homing
   direction map. 31/31 tests pass.

Co-Authored-By: Claude Fable 5 <noreply@anthropic.com>
Claude-Session: https://claude.ai/code/session_0164ttHi9eFxn6JBT957rEqQ

File: ros2_ws/src/nova_description/urdf/leg.macro.xacro (robot description, xacro)
@@ -19,5 +19,9 @@
       <origin xyz="${mount_x} ${mount_y} ${mount_z}" rpy="0 0 0"/>
       <axis xyz="1 0 0"/>
-      <limit lower="${-haa_range}" upper="${haa_range}"
+      <!-- asymmetric gate ROM: inboard 15 / outboard 40 (chassis gate).
+           +roll swings feet toward +y: inboard for RIGHT (reflect -1),
+           outboard for LEFT (reflect +1). -->
+      <limit lower="${-haa_in if reflect == 1 else -haa_out}"
+             upper="${haa_out if reflect == 1 else haa_in}"
              effort="${eff_hip}" velocity="${vel_servo}"/>
     </joint>
@@ -38,5 +42,7 @@
       <origin xyz="${hip_to_upper_x} ${reflect*hip_to_upper_y} ${hip_to_upper_z}" rpy="0 0 0"/>
       <axis xyz="0 1 0"/>
-      <limit lower="${-hfe_range}" upper="${hfe_range}"
+      <!-- gate ROM: away-trunk -86 .. toward-trunk +50 (sign mapping
+           ⚠ VERIFY IN SIM — see nova.urdf.xacro) -->
+      <limit lower="${-hfe_ext}" upper="${hfe_fold}"
              effort="${eff_leg}" velocity="${vel_servo}"/>
     </joint>

File: ros2_ws/src/nova_description/urdf/nova.urdf.xacro (robot description, xacro)
@@ -20,6 +20,18 @@
   <xacro:property name="eff_leg"  value="1.8"/>
   <xacro:property name="vel_servo" value="6.0"/>
-  <xacro:property name="haa_range" value="0.7"/>   <!-- TODO-CAD mechanical travel -->
-  <xacro:property name="hfe_range" value="1.5"/>   <!-- TODO-CAD -->
+  <!-- ROM = the CAD fit gates (chassis check_fit crouch sweep = authority,
+       2026-07-06; replaces the TODO-CAD placeholders):
+       haa: OUTBOARD 40 sw / INBOARD 15 sw (belly-pack contact from ~18
+            inboard at any fold >= 30). Inboard for a RIGHT leg (y<0) =
+            +roll about the +x axis; LEFT = -roll — per-side via reflect
+            in leg.macro.
+       hfe: toward-trunk fold +50 sw (tibia flank grazes the riser skirt
+            from ~+55) / away-trunk -86 sw. ⚠ SIGN MAPPING gate->URDF
+            assumed +hfe = toward-trunk, same for all four legs (knees
+            translated, one convention) — VERIFY IN SIM before gait. -->
+  <xacro:property name="haa_in"   value="0.262"/>  <!-- 15 deg inboard -->
+  <xacro:property name="haa_out"  value="0.698"/>  <!-- 40 deg outboard -->
+  <xacro:property name="hfe_fold" value="0.873"/>  <!-- +50 toward trunk -->
+  <xacro:property name="hfe_ext"  value="1.501"/>  <!-- -86 away -->
   <xacro:property name="kfe_range" value="1.9"/>   <!-- sweep-gate: mech stop ~118 deg (tibia flank vs fork throat); 109 sw = margin. Deep-sit = v7 offset-plane option -->
   <!-- ===================== link offsets (m) ===================== -->
@@ -56,10 +68,18 @@
   <xacro:property name="lower_to_foot_z" value="-0.1290"/> <!-- MEASURED tibia length -->
   <!-- ===================== masses (kg) ===================== -->
-  <!-- TODO-CAD: weigh / compute from CAD. STS3215 ≈ 0.06 kg each. -->
-  <xacro:property name="m_base"  value="1.2"/>
-  <xacro:property name="m_hip"   value="0.12"/>
-  <xacro:property name="m_upper" value="0.16"/>
-  <xacro:property name="m_lower" value="0.08"/>
-  <xacro:property name="m_foot"  value="0.02"/>
+  <!-- CAD-volume estimates 2026-07-06 (leg_v6 STL volume x 1.17 g/cm3
+       PA6-CF x 0.7 infill factor) + STS3215 0.055 each; servo rides the
+       link whose pocket houses it (coax=HAA, femur=HFE, tibia=KFE).
+       hip = coax 27g + servo; upper = femur 61 + knee_arm 6 + servo +
+       hardware; lower = tibia 70 + servo + strap; foot = TPU shoe.
+       ⚠ ESTIMATES — weigh the printed set at the next print batch
+       (backlog #5) and replace. m_base = mass budget 4.2 minus legs
+       (trunk+riser+shoulders+Jetson+battery+boards+L2+D456), the
+       roughest number here. -->
+  <xacro:property name="m_base"  value="2.83"/>
+  <xacro:property name="m_hip"   value="0.082"/>
+  <xacro:property name="m_upper" value="0.127"/>
+  <xacro:property name="m_lower" value="0.130"/>
+  <xacro:property name="m_foot"  value="0.005"/>
   <!-- crude box inertia helper (TODO-CAD: replace with real tensors) -->
   <xacro:macro name="link_inertial" params="mass">

Commit message: chassis: integrated forward HEAD (D456 tilted face + L2 crown), retire mast+periscope
Replace the two front sensor parts (l2_mast periscope-era mast + d456_head
periscope) with ONE head.scad that carries BOTH sensors: the RealSense D456
as a 27-degree DOWN-tilted "face" forward of the chassis (back-face ctr
70,0,105.5) and the Unitree L2 as a "crown" on top (optical z~154). This
fixes the periscope's near-ground occlusion — the trunk front no longer cuts
the bottom of the camera view, because the camera sits forward of the front
wall (x63.5) and looks down.

head_study.py (the placement proof) verifies against the REAL swept front-leg
cloud: D456 body x63.4..99.7 z80.8..118.4 clears the front-leg sweep with 0
hits, the deck-ext fins (+1.2 over the fin top), and stays inside x100; L2
360-deg ring clear (camera top 36 below), rear-down cone blind only below
-83deg (Jetson case, v1-accepted), and the D456 no longer clips the L2 forward
cone (the periscope clipped ~3.5deg). CoM fore-aft shift ~= 0 (L2 kept at
x53.5; the tilt pulls the D456 centroid ~1mm rearward).

Feasibility REQUIRES capping FRONT hfe forward protraction at -50 (was -86):
a front leg reaching -86 forward sweeps the head volume. Wired leg-dependent:
URDF hfe_ext_front (front) vs hfe_ext (rear) via leg[0]=='F' in leg.macro;
limits.py note; check_fit.py HEAD case uses hfe_lo -50 front / -86 rear. Rear
legs keep -86. Fold (+50) unchanged. Front -50 is still a strong stride (gait
uses -30..-50).

- head.scad: rear L2 tower (reuses mast deck base + 13x11 bore + 4x M3 22.5
  crown, seat raised to 122 to clear the tilted face) + front D456 face (stem
  through the flange notch to the wall row, tilted plate on the 2x M3 @94.4
  centerline + z-slot, USB-C window->stem channel->wall grommet). Watertight,
  single body, 39cm3.
- check_fit.py: fused mast(7)+D456(8) cases into one HEAD case (tilted-OBB
  camera helper + seated-L2 box); front-hfe -50 cap in the crouch sweep;
  case-10 + static asserts updated to the raised crown (118/122).
- riser_bay.scad: relabel the two anchor patterns (deck L2-column base +
  front-wall camera register) as the single head mount; geometry UNCHANGED,
  gate stays clean.
- l2_mast.scad / d456_head.scad: RETIRED headers -> head.scad; removed from
  build_all + preview; stale STLs deleted.
- dimensions.md + chassis/README.md: retire mast/periscope rows, add head +
  the front-hfe -50 rationale. Fuse block remains an OPEN assembly-time item.

Both gates clean (chassis check_fit exit 0, leg_v6 gate 0 CUTs); mesh_health
green; nova_ops + nova_locomotion URDF/limits tests pass.

Co-Authored-By: Claude Fable 5 <noreply@anthropic.com>
Claude-Session: https://claude.ai/code/session_0164ttHi9eFxn6JBT957rEqQ

File: ros2_ws/src/nova_description/urdf/leg.macro.xacro (robot description, xacro)
@@ -42,7 +42,9 @@
       <origin xyz="${hip_to_upper_x} ${reflect*hip_to_upper_y} ${hip_to_upper_z}" rpy="0 0 0"/>
       <axis xyz="0 1 0"/>
-      <!-- gate ROM: away-trunk -86 .. toward-trunk +50 (sign mapping
-           ⚠ VERIFY IN SIM — see nova.urdf.xacro) -->
-      <limit lower="${-hfe_ext}" upper="${hfe_fold}"
+      <!-- gate ROM: toward-trunk +50 (both) .. away-trunk -50 FRONT / -86 REAR.
+           FRONT protraction capped -50 for the forward head (2026-07-07; sign
+           mapping ⚠ VERIFY IN SIM — see nova.urdf.xacro). -->
+      <limit lower="${-hfe_ext_front if leg[0] == 'F' else -hfe_ext}"
+             upper="${hfe_fold}"
              effort="${eff_leg}" velocity="${vel_servo}"/>
     </joint>

File: ros2_ws/src/nova_description/urdf/nova.urdf.xacro (robot description, xacro)
@@ -27,11 +27,17 @@
             in leg.macro.
        hfe: toward-trunk fold +50 sw (tibia flank grazes the riser skirt
-            from ~+55) / away-trunk -86 sw. ⚠ SIGN MAPPING gate->URDF
-            assumed +hfe = toward-trunk, same for all four legs (knees
-            translated, one convention) — VERIFY IN SIM before gait. -->
+            from ~+55), BOTH ends. Away-trunk (forward protraction) is now
+            LEG-DEPENDENT (head clearance, 2026-07-07): FRONT legs cap at
+            -50 (the forward HEAD occupies x70..100 z80..120; front legs
+            reaching -86 forward hit the D456 face / L2 crown — chassis
+            check_fit HEAD case), REAR legs keep -86. Front -50 is still a
+            strong stride (gait uses -30..-50; kfe-109 chord still reaches).
+            ⚠ SIGN MAPPING gate->URDF assumed +hfe = toward-trunk, same for
+            all four legs (knees translated, one convention) — VERIFY IN SIM. -->
   <xacro:property name="haa_in"   value="0.262"/>  <!-- 15 deg inboard -->
   <xacro:property name="haa_out"  value="0.698"/>  <!-- 40 deg outboard -->
-  <xacro:property name="hfe_fold" value="0.873"/>  <!-- +50 toward trunk -->
-  <xacro:property name="hfe_ext"  value="1.501"/>  <!-- -86 away -->
+  <xacro:property name="hfe_fold" value="0.873"/>  <!-- +50 toward trunk (both) -->
+  <xacro:property name="hfe_ext"       value="1.501"/>  <!-- -86 away, REAR legs -->
+  <xacro:property name="hfe_ext_front" value="0.873"/>  <!-- -50 away, FRONT legs (head cap) -->
   <xacro:property name="kfe_range" value="1.9"/>   <!-- sweep-gate: mech stop ~118 deg (tibia flank vs fork throat); 109 sw = margin. Deep-sit = v7 offset-plane option -->
   <!-- ===================== link offsets (m) ===================== -->

Commit message: fix(#47): correct stale front hfe head-clearance cap (-50 was wrong) + clamp
Decision was "measure the true cap, then clamp + retune" — the measurement
flipped the premise. head_cap_sweep.py (new, reuses check_fit's validated FR-hip
transforms + a positive control that reproduces the known riser graze before
trusting any negative) swept the front leg vs the real head assembly (head, l2
_adapter, ears, l2_ref/d456 convex hulls) across hfe -35..-95 x full kfe x haa:
ZERO leg<->head contact anywhere, min clearance 32.1mm (legal ROM), 19.5mm even
at the not-yet-legal 40deg outboard cap. The real front limit is the leg's OWN
self-collision (~93deg mech / 86deg sw, leg_v6 LA-19) — same as the rear leg.

Root cause: the -50deg front cap was set 2026-07-07 (the day the head moved
FORWARD onto the shoulder deck) and never re-validated — stale, not
conservative. The chassis gate's own head-vs-front-leg window (|y|<40) was a
silent no-op the whole time (front-leg cloud never drops below y~21).

- hfe_ext_front -50 -> -86deg (= hfe_ext, rear) in nova.urdf.xacro + leg.macro
  comment + limits.py _thigh_flexion + leg_ik.LegParams.hfe_min_front.
- Runtime clamp in leg_ik.solve_side() (new leg= param) — the single choke point
  all commanded poses funnel through (stand.pose_for + controller.gait_pose) —
  backstops front hfe to [hfe_min_front, hfe_max] regardless of gait source.
- No gait retune needed: trot/crawl/raibert/body-pose worst-case front hfe is
  -57..-66deg, well inside -86. RESTORED stand.py crouch/lie to their original
  0.150/0.140 depths (LA-13 had shrunk them to 0.176/0.172 against the stale
  cap) — recovers full E-stop-sim fold depth; kfe is the real binding constraint
  there (~1deg margin at lie).
- Tests: dropped the "don't pass leg=" workarounds, assert real legality, added
  a solve_side front-clamp test. 144 passed (preflight excluded — needs rclpy/
  Jetson, off-bench skip per /rostest).

Supersedes the interim in d62026b. Closes #47.

Co-Authored-By: Claude Opus 4.8 (1M context) <noreply@anthropic.com>
Claude-Session: https://claude.ai/code/session_0144vPbdpqh96UgWG8ybLgSs

File: ros2_ws/src/nova_description/urdf/leg.macro.xacro (robot description, xacro)
@@ -42,7 +42,10 @@
       <origin xyz="${hip_to_upper_x} ${reflect*hip_to_upper_y} ${hip_to_upper_z}" rpy="0 0 0"/>
       <axis xyz="0 1 0"/>
-      <!-- gate ROM: toward-trunk +50 (both) .. away-trunk -50 FRONT / -86 REAR.
-           FRONT protraction capped -50 for the forward head (2026-07-07; sign
-           mapping ⚠ VERIFY IN SIM — see nova.urdf.xacro). -->
+      <!-- gate ROM: toward-trunk +50 (both) .. away-trunk -86 (both — #47
+           MEASURED 2026-07-11: front head clearance is not the binding
+           constraint, leg self-collision is; see nova.urdf.xacro's
+           hfe_ext_front comment). Still keyed per-leg via hfe_ext_front so
+           a future head-position change only needs one property changed
+           (sign mapping ⚠ VERIFY IN SIM — see nova.urdf.xacro). -->
       <limit lower="${-hfe_ext_front if leg[0] == 'F' else -hfe_ext}"
              upper="${hfe_fold}"

File: ros2_ws/src/nova_description/urdf/nova.urdf.xacro (robot description, xacro)
@@ -27,10 +27,26 @@
             in leg.macro.
        hfe: toward-trunk fold +50 sw (tibia flank grazes the riser skirt
-            from ~+55), BOTH ends. Away-trunk (forward protraction) is now
-            LEG-DEPENDENT (head clearance, 2026-07-07): FRONT legs cap at
-            -50 (the forward HEAD occupies x70..100 z80..120; front legs
-            reaching -86 forward hit the D456 face / L2 crown — chassis
-            check_fit HEAD case), REAR legs keep -86. Front -50 is still a
-            strong stride (gait uses -30..-50; kfe-109 chord still reaches).
+            from ~+55), BOTH ends. Away-trunk (forward protraction):
+            #47 (2026-07-11, MEASURED — hardware/cad/chassis/
+            head_cap_sweep.py): a FINE hfe sweep of the FRONT leg
+            (femur_R+knee_arm+tibia_R+knee_bumper+shoe) vs the REAL head
+            assembly (head.stl, l2_adapter.stl, head_ear.stl/_L.stl, plus
+            convex hulls of the non-watertight l2_ref.stl/d456_ref.stl)
+            found ZERO contact anywhere in the front leg's structurally-
+            reachable hfe range (-35..-95, i.e. past leg_v6's own measured
+            ~93deg self-collision mech stop) at any kfe/haa combo —
+            min clearance ~34mm at today's legal haa (<=15deg), ~20mm even
+            at the not-yet-unlocked 40deg outboard cap. The -50 value here
+            (set 2026-07-07, the SAME day the head moved forward onto the
+            front-shoulder deck — chassis/check_fit.py HEAD geometry
+            comments) was never re-validated after that move: it was
+            STALE, not conservative-by-design. FRONT and REAR now share
+            the SAME real governing constraint instead — leg_v6/
+            check_fit.py's own hip-pitch self-collision sweep (LA-19:
+            clean to 92.5deg, first contact 93deg) — so hfe_ext_front ==
+            hfe_ext (86deg sw, the same 7deg margin already used
+            everywhere else in this file). Kept as a separate property
+            (not deleted/merged into hfe_ext) so a future head-position
+            change has one obvious knob to retighten.
             ⚠ SIGN MAPPING gate->URDF assumed +hfe = toward-trunk, same for
             all four legs (knees translated, one convention) — VERIFY IN SIM. -->
@@ -39,5 +55,5 @@
   <xacro:property name="hfe_fold" value="0.873"/>  <!-- +50 toward trunk (both) -->
   <xacro:property name="hfe_ext"       value="1.501"/>  <!-- -86 away, REAR legs -->
-  <xacro:property name="hfe_ext_front" value="0.873"/>  <!-- -50 away, FRONT legs (head cap) -->
+  <xacro:property name="hfe_ext_front" value="1.501"/>  <!-- -86 away, FRONT legs — #47: head clearance is NOT the binding constraint (measured), leg self-collision (LA-19, 93deg) is; matches hfe_ext -->
   <xacro:property name="kfe_range" value="1.9"/>   <!-- sweep-gate: mech stop ~118 deg (tibia flank vs fork throat); 109 sw = margin. Deep-sit = v7 offset-plane option -->
   <!-- ===================== link offsets (m) ===================== -->
