Commit message: nova_description: real per-link inertials from CAD (replaces placeholders)
The URDF shipped crude isotropic inertials (ixx=iyy=izz=mass*1e-3, CoM at
the joint) — fine for RViz, wrong for MJX/Isaac RL. Replace with real
mass / CoM / anisotropic inertia tensors computed from the leg_v6 meshes +
embedded STS3215 servos.

- tools/compute_inertials.py — loads each real part (coax/femur+knee_arm/
  tibia/shoe) at effective PA6-CF density (1.17 g/cm3 x 0.70 infill) + a
  60 g servo box per pocket, combines via parallel-axis, maps STL frame ->
  URDF link frame. Frame maps validated against the URDF's own landmarks
  (femur STL (106.9,0,0) -> link (0,0,-0.1069); tibia foot-jog sign).
- nova.urdf.xacro / leg.macro.xacro — per-link inertial macros (hip/upper/
  lower/foot + a base box), y-terms mirrored L/R via reflect.

Computed masses validate vs the old estimates (hip .087 vs .082, upper
.131 vs .127, lower .131 vs .130 kg) and the anisotropy is physical (izz
smallest = about each leg's long axis). Both xacro files parse well-formed;
urdf_sync test green.

⚠ PROVISIONAL — refine by measurement (backlog #5): weigh each printed
link, rescale its <inertial> by measured/computed mass (linear; CoM
unchanged). Servo-at-shell-centroid + L/R y-sign flagged to verify in sim.
base_link stays payload-dominated (~2.8 kg); box inertia + assembled-CoM
still owed.

Co-Authored-By: Claude Opus 4.8 (1M context) <noreply@anthropic.com>
Claude-Session: https://claude.ai/code/session_01PfnMkwGYyVsyLfTtBhHzYb

File: ros2_ws/src/nova_description/urdf/leg.macro.xacro (robot description, xacro)
@@ -34,5 +34,5 @@
         <geometry><mesh filename="package://nova_description/meshes/SM3_Frame_${side}Coax.stl" scale="0.001 0.001 0.001"/></geometry>
       </collision>
-      <xacro:link_inertial mass="${m_hip}"/>
+      <xacro:hip_inertial reflect="${reflect}"/>
     </link>
     <!-- ===== HFE : hip -> upper (femur) ===== -->
@@ -59,5 +59,5 @@
         <geometry><mesh filename="package://nova_description/meshes/SM3_Frame_${side}Femur.stl" scale="0.001 0.001 0.001"/></geometry>
       </collision>
-      <xacro:link_inertial mass="${m_upper}"/>
+      <xacro:upper_inertial reflect="${reflect}"/>
     </link>
     <!-- ===== KFE : upper -> lower (tibia) ===== -->
@@ -77,5 +77,5 @@
         <geometry><mesh filename="package://nova_description/meshes/SM3_Frame_${side}Tibia.stl" scale="0.001 0.001 0.001"/></geometry>
       </collision>
-      <xacro:link_inertial mass="${m_lower}"/>
+      <xacro:lower_inertial reflect="${reflect}"/>
     </link>
     <!-- ===== foot (fixed) ===== -->
@@ -90,5 +90,5 @@
       </visual>
       <collision><geometry><sphere radius="0.012"/></geometry></collision>
-      <xacro:link_inertial mass="${m_foot}"/>
+      <xacro:foot_inertial reflect="${reflect}"/>
     </link>
   </xacro:macro>

File: ros2_ws/src/nova_description/urdf/nova.urdf.xacro (robot description, xacro)
@@ -89,25 +89,63 @@
   <xacro:property name="lower_to_foot_x" value="0.0"/>
   <xacro:property name="lower_to_foot_z" value="-0.1290"/> <!-- MEASURED tibia length -->
-  <!-- ===================== masses (kg) ===================== -->
-  <!-- CAD-volume estimates 2026-07-06 (leg_v6 STL volume x 1.17 g/cm3
-       PA6-CF x 0.7 infill factor) + STS3215 0.055 each; servo rides the
-       link whose pocket houses it (coax=HAA, femur=HFE, tibia=KFE).
-       hip = coax 27g + servo; upper = femur 61 + knee_arm 6 + servo +
-       hardware; lower = tibia 70 + servo + strap; foot = TPU shoe.
-       ⚠ ESTIMATES — weigh the printed set at the next print batch
-       (backlog #5) and replace. m_base = mass budget 4.2 minus legs
-       (trunk+riser+shoulders+Jetson+battery+boards+L2+D456), the
-       roughest number here. -->
+  <!-- ===================== masses + inertials ===================== -->
+  <!-- COMPUTED 2026-07-13 from the REAL leg_v6 meshes + embedded STS3215 servos
+       (tools/compute_inertials.py): full mass / CoM / anisotropic inertia tensor
+       per link, mapped into each URDF link frame (frame maps validated vs the
+       URDF's own landmarks — femur STL (106.9,0,0) -> link (0,0,-0.1069)).
+       Replaces the old isotropic mass*1e-3 placeholders.
+       ⚠ PROVISIONAL — REFINE BY MEASUREMENT (backlog #5). Mass = solid mesh
+       volume x effective PA6-CF density (1.17 g/cm3 x 0.70 infill) + a 60 g
+       servo box at each pocket. When you WEIGH each printed link, rescale that
+       link's whole <inertial> by measured_mass/computed_mass (CoM unchanged;
+       inertia scales linearly with mass) — one ratio absorbs the density error.
+       ⚠ Servo modeled at the shell centroid; ⚠ LEFT/RIGHT y-sign mirrored via
+       `reflect` (yf=-reflect on com_y/ixy/iyz) — VERIFY THE SIGN IN SIM (matches
+       this file's other gate->URDF sign caveats). base_link stays payload-
+       dominated (~2.8 kg trunk+Jetson+battery+boards+L2/D456); box inertia +
+       measured-CoM refinement still owed.
+       Computed right-leg masses: hip 0.087 upper 0.131 lower 0.131 foot 0.004
+       (vs the old 0.082/0.127/0.130/0.005 estimates — within ~6%). -->
   <xacro:property name="m_base"  value="2.83"/>
-  <xacro:property name="m_hip"   value="0.082"/>
-  <xacro:property name="m_upper" value="0.127"/>
-  <xacro:property name="m_lower" value="0.130"/>
-  <xacro:property name="m_foot"  value="0.005"/>
-  <!-- crude box inertia helper (TODO-CAD: replace with real tensors) -->
-  <xacro:macro name="link_inertial" params="mass">
+  <!-- base_link: trunk envelope box inertia at m_base (payload-dominated,
+       CoM at the geometric center — refine with the assembled-stack CoM). -->
+  <xacro:macro name="base_inertial" params="">
     <inertial>
       <origin xyz="0 0 0" rpy="0 0 0"/>
-      <mass value="${mass}"/>
-      <inertia ixx="${mass*1e-3}" iyy="${mass*1e-3}" izz="${mass*1e-3}"
+      <mass value="${m_base}"/>
+      <inertia ixx="8.7e-03" iyy="2.46e-02" izz="2.65e-02"
+               ixy="0" ixz="0" iyz="0"/>
+    </inertial>
+  </xacro:macro>
+  <!-- per-link real inertials (RIGHT-leg values; yf mirrors y-terms for LEFT) -->
+  <xacro:macro name="hip_inertial" params="reflect">
+    <inertial>
+      <origin xyz="0.00710 ${-reflect*0.02004} 0.00497" rpy="0 0 0"/>
+      <mass value="0.0873"/>
+      <inertia ixx="4.452e-05" iyy="2.275e-05" izz="3.552e-05"
+               ixy="${-reflect*-2.20e-06}" ixz="8.41e-07" iyz="${-reflect*3.81e-06}"/>
+    </inertial>
+  </xacro:macro>
+  <xacro:macro name="upper_inertial" params="reflect">
+    <inertial>
+      <origin xyz="0.00000 ${-reflect*-0.00653} -0.05067" rpy="0 0 0"/>
+      <mass value="0.1313"/>
+      <inertia ixx="8.366e-05" iyy="7.473e-05" izz="2.907e-05"
+               ixy="${-reflect*-9.47e-10}" ixz="-4.45e-10" iyz="${-reflect*-4.08e-06}"/>
+    </inertial>
+  </xacro:macro>
+  <xacro:macro name="lower_inertial" params="reflect">
+    <inertial>
+      <origin xyz="-0.00054 ${-reflect*-0.01010} -0.06558" rpy="0 0 0"/>
+      <mass value="0.1312"/>
+      <inertia ixx="1.333e-04" iyy="1.225e-04" izz="2.809e-05"
+               ixy="${-reflect*-7.87e-07}" ixz="-1.94e-06" iyz="${-reflect*-1.87e-05}"/>
+    </inertial>
+  </xacro:macro>
+  <xacro:macro name="foot_inertial" params="reflect">
+    <inertial>
+      <origin xyz="0 0 0" rpy="0 0 0"/>
+      <mass value="0.0039"/>
+      <inertia ixx="2.116e-07" iyy="5.602e-07" izz="5.763e-07"
                ixy="0" ixz="0" iyz="0"/>
     </inertial>
@@ -122,5 +160,5 @@
       <geometry><mesh filename="package://nova_description/meshes/SM3_Frame_ChassisTrunk.stl" scale="0.001 0.001 0.001"/></geometry>
     </collision>
-    <xacro:link_inertial mass="${m_base}"/>
+    <xacro:base_inertial/>
   </link>
   <!-- ===================== 4 legs =====================

Commit message: model: put the pitch axes where leg_v6 actually builds them (#165)
body_half_x 0.1412 + hip_to_upper_x 0.0 was a STOCK-assembly pair. On stock it
is exact: the haa axis is fore-aft parallel, so sliding the hip origin ALONG it
is a kinematic no-op, and putting that origin at the hfe station reproduces the
geometry. leg_v6 broke the identity — shoulder.scad fixes the haa station at
+-141.2 (trunk end face +-63.5 + 77.7 flange) and coax.scad puts the hfe axis
11.6 mm TOWARD THE TRUNK of it at both ends, once the rear crossmember is
correctly yawed 180 deg (#163). Real pitch spacing is 259.2, not 282.4, so the
modeled stance was 23.2 mm (8.9%) longer fore-aft than the robot — on a
platform where CoM offsets are argued at +-5 mm.

Fixed in the form that describes the hardware literally (the issue's
recommendation): body_half_x stays 0.1412 because that IS the haa station, and
the femur is offset 11.6 mm inboard of it. The alternative (body_half_x ->
0.1296) moves the hip JOINTS instead — same hip-relative leg chain, different
base_link-relative stance. That is a different robot, not a different spelling.

PER END, NOT PER SIDE: toward-the-trunk is -x at the front and +x at the rear,
so leg.macro.xacro keys the sign off leg[0] (as the hfe extension limit already
does) and build_mjcf keys it off sx. A reflect-style per-SIDE sign would look
right on the left legs and put both rear hips on the far side of their own hip
station — #163 again.

- nova.urdf.xacro + leg.macro.xacro, sim/nova_mjx/build_mjcf.py, regenerated
  sim/nova_mjx/nova.xml (pitch axes now +-0.1296).
- test_urdf_sync gains three cross-seam tests reading the station from
  check_fit.py HIP_FA and coax.scad HFE_Y — the CAD constants, not a number
  retyped into the test — plus a front/rear sign check as the negative control
  for the per-side mistake. Both station tests fail against the old geometry;
  verified by reverting.
- dimensions.md "Hip grid" note resolved.

Link frames do not move relative to their own parents, so compute_inertials.py
output is unaffected and is not re-run here.

217 pass.

NOT in scope, found while doing this: body_pose.hip_mounts anchors the leg
plane at the HAA station and LegParams carries no fore-aft haa->hfe term, so
the locomotion stack still assumes the pre-v6 identity. Filed separately —
changing it moves commanded foot targets, which is a gait-lane call.

Co-Authored-By: Claude Opus 5 (1M context) <noreply@anthropic.com>
Claude-Session: https://claude.ai/code/session_017cpi4kYCP39PAeE7d48Qu2

File: ros2_ws/src/nova_description/urdf/leg.macro.xacro (robot description, xacro)
@@ -40,5 +40,10 @@
       <parent link="${leg}_hip"/>
       <child  link="${leg}_upper"/>
-      <origin xyz="${hip_to_upper_x} ${reflect*hip_to_upper_y} ${hip_to_upper_z}" rpy="0 0 0"/>
+      <!-- hip_to_upper_x is a MAGNITUDE; the hfe axis sits that far TOWARD THE
+           TRUNK of the haa station (#165). That is -x at the front and +x at
+           the rear, so the sign is keyed per END (leg[0]) exactly like the hfe
+           extension limit below — NOT per side via reflect, which would put
+           both rear hips on the wrong side of their own hip station. -->
+      <origin xyz="${hip_to_upper_x if leg[0] == 'R' else -hip_to_upper_x} ${reflect*hip_to_upper_y} ${hip_to_upper_z}" rpy="0 0 0"/>
       <axis xyz="0 1 0"/>
       <!-- gate ROM: toward-trunk +50 (both) .. away-trunk -86 (both — #47

File: ros2_ws/src/nova_description/urdf/nova.urdf.xacro (robot description, xacro)
@@ -65,21 +65,34 @@
        the tibia S-curve puts the foot 30.5 mm outboard of kfe.
        Total haa->foot lateral = 64.3 mm = LegParams.hip_offset. -->
-  <!-- ⚠ OPEN (CAD review 2026-07-26): body_half_x + hip_to_upper_x below are a
-       STOCK-assembly pair. 141.2 is the stock HFE-axis fore-aft station, which
-       is why hip_to_upper_x = 0 is exact for stock (the haa axis is fore-aft
-       parallel, so its own station along that axis is a kinematic no-op).
-       leg_v6 moved it: shoulder.scad puts the haa station at ±141.2 (trunk end
-       face ±63.5 + 77.7 flange) and coax.scad puts the hfe axis 11.6 mm TOWARD
-       THE TRUNK of it, at both ends -> real pitch-axis spacing 259.2, not
-       282.4. So this model's stance is 23.2 mm longer fore-aft than the built
-       robot (same error in sim/nova_mjx/build_mjcf.py MOUNT/HAA_TO_HFE).
-       Fix is either body_half_x 0.1296 or hip_to_upper_x ∓0.0116 — NOT changed
-       here: it shifts every trained policy's geometry and is a B2/gait-lane
-       call. Details: hardware/cad/dimensions.md "Hip grid" +
-       docs/cad-review-2026-07-26.md §2. -->
-  <xacro:property name="body_half_x" value="0.1412"/> <!-- MEASURED half hip-grid length (⚠ stock hfe station, see above) -->
+  <!-- HIP GRID, fixed 2026-07-27 (#165). These two were a STOCK-assembly pair:
+       141.2 is the stock HFE-axis fore-aft station, and on stock that made
+       hip_to_upper_x = 0 exact — the haa axis is fore-aft parallel, so sliding
+       the hip origin ALONG it is a kinematic no-op, and putting the origin at
+       the hfe station reproduces the geometry.
+       leg_v6 broke that identity: shoulder.scad fixes the haa station at ±141.2
+       (trunk end face ±63.5 + 77.7 flange) and coax.scad puts the hfe axis
+       11.6 mm TOWARD THE TRUNK of it — at BOTH ends, once the rear crossmember
+       is correctly yawed 180 deg (#163). Real pitch-axis spacing is 259.2, not
+       282.4, so the model's stance was 23.2 mm (8.9%) longer fore-aft than the
+       robot, on a platform where CoM offsets are argued at ±5 mm.
+       Fixed in the form that describes the hardware literally: the haa station
+       really IS ±141.2 (body_half_x unchanged) and the femur really IS 11.6 mm
+       inboard of it. The alternative (body_half_x -> 0.1296) would have moved
+       the hip JOINTS instead, which is a different robot — same foot-relative-
+       to-hip chain, different base_link-relative stance.
+       PER END, NOT PER SIDE: toward-the-trunk is -x at the front and +x at the
+       rear, so leg.macro.xacro keys the sign off leg[0], the same way the hfe
+       extension limit already does. A `reflect`-style per-SIDE sign would put
+       both rear hips on the wrong side of their own hip station.
+       Link frames do not move relative to their own parents' inertia frames, so
+       compute_inertials.py output is unaffected. Mirrored in
+       sim/nova_mjx/build_mjcf.py (HAA_TO_HFE[0]).
+       Refs: hardware/cad/dimensions.md "Hip grid", docs/cad-review-2026-07-26.md
+       §2, #163/#164. -->
+  <xacro:property name="body_half_x" value="0.1412"/> <!-- MEASURED half hip-grid length (haa station, shoulder.scad) -->
   <xacro:property name="body_half_y" value="0.0390"/> <!-- MEASURED half hip-grid width  -->
   <xacro:property name="mount_z"     value="0.0380"/> <!-- hip row above chassis-mesh origin; ⚠ REVIEW-visual (trunk-node bbox polluted by children) -->
-  <xacro:property name="hip_to_upper_x" value="0.0"/>
+  <!-- MAGNITUDE. Sign is applied per END in leg.macro.xacro (toward trunk). -->
+  <xacro:property name="hip_to_upper_x" value="0.0116"/> <!-- haa axis -> hfe axis, along the trunk axis (coax.scad HFE_Y) -->
   <!-- v6 legs (leg_v6/): femur mid-plane 33.8 from haa (coax yoke), femur/
        tibia coplanar (0), toe tab jogs 30.5 OUTBOARD (stock stance: straight
